Commit message: update elfin5.urdf.xacro for inertial info

File: elfin_description/urdf/elfin5.urdf.xacro (robot description, xacro)
@@ -5,4 +5,5 @@
   <xacro:include filename="$(find elfin_description)/urdf/elfin_transmission.xacro" />
   <xacro:property name="PI" value="3.1415926535897931"/>
+  <xacro:property name="density" value="3.09"/>
   <link name="world"/>
   <joint name="world_base" type="fixed">
@@ -29,11 +30,11 @@
     <inertial>
       <origin
-        xyz="0.000220821977982989 0.0255290818849933 -0.00134044659901771"
-        rpy="0 0 0" />
-      <mass value="0.05"/>
-      <inertia
-	  ixx="0.001" ixy="0.0" ixz="0.0"
-	  iyy="0.001" iyz="0.0"
-	  izz="0.001"/>
+        xyz="0.000209 0.001319 0.025619"
+        rpy="0 0 0" />
+      <mass value="${0.690521*density}"/>
+      <inertia
+	  ixx="${0.00130611*density}" ixy="${0.0000568*density}" ixz="${0.00000189*density}"
+	  iyy="${0.00134467*density}" iyz="${0.00001095*density}"
+	  izz="${0.00229139*density}"/>
     </inertial>
     <visual>
@@ -62,11 +63,11 @@
     <inertial>
       <origin
-        xyz="-0.0218141046310325 0.138891728726282 1.31241816829816E-05"
-        rpy="0 0 0" />
-      <mass value="0.05"/>
-      <inertia
-	  ixx="0.001" ixy="0.0" ixz="0.0"
-	  iyy="0.001" iyz="0.0"
-	  izz="0.001"/>
+        xyz="-0.0217491 0.1389011 0.0000125"
+        rpy="0 0 0" />
+      <mass value="${2.576772*density}"/>
+      <inertia
+	  ixx="${0.01298966*density}" ixy="${0.00287966*density}" ixz="${-0.000001*density}"
+	  iyy="${0.00721115*density}" iyz="${-0.00000052*density}"
+	  izz="${0.01532713*density}"/>
     </inertial>
     <visual>
@@ -113,11 +114,11 @@
     <inertial>
       <origin
-        xyz="-0.0524295669840444 0.158140141659462 -1.74919824000372E-06"
-        rpy="0 0 0" />
-      <mass value="0.05"/>
-      <inertia
-	  ixx="0.001" ixy="0.0" ixz="0.0"
-	  iyy="0.001" iyz="0.0"
-	  izz="0.001"/>
+        xyz="-0.0522485 0.1580101 -0.0000003"
+        rpy="0 0 0" />
+      <mass value="${1.208607*density}"/>
+      <inertia
+	  ixx="${0.02975970*density}" ixy="${-0.00126441*density}" ixz="${-0.00000024*density}"
+	  iyy="${0.00168156*density}" iyz="${-0.0000021*density}"
+	  izz="${0.02944694*density}"/>
     </inertial>
     <visual>
@@ -164,11 +165,11 @@
     <inertial>
       <origin
-        xyz="0.0586561082766824 -0.0414791884757505 -9.80549635387022E-06"
-        rpy="0 0 0" />
-      <mass value="0.05"/>
-      <inertia
-	  ixx="0.001" ixy="0.0" ixz="0.0"
-	  iyy="0.001" iyz="0.0"
-	  izz="0.001"/>
+        xyz="0.0587091 -0.0414608 -0.0000210"
+        rpy="0 0 0" />
+      <mass value="${1.525883*density}"/>
+      <inertia
+	  ixx="${0.00527835*density}" ixy="${0.00124150*density}" ixz="${-0.00000018*density}"
+	  iyy="${0.00317861*density}" iyz="${-0.00000067*density}"
+	  izz="${0.00652527*density}"/>
     </inertial>
     <visual>
@@ -215,11 +216,11 @@
     <inertial>
       <origin
-        xyz="-0.0589525602581192 0.143654952750886 -4.64578965075454E-05"
-        rpy="0 0 0" />
-      <mass value="0.05"/>
-      <inertia
-	  ixx="0.001" ixy="0.0" ixz="0.0"
-	  iyy="0.001" iyz="0.0"
-	  izz="0.001"/>
+        xyz="-0.0587964 0.1436154 -0.0000478"
+        rpy="0 0 0" />
+      <mass value="${0.475026*density}"/>
+      <inertia
+	  ixx="${0.00542441*density}" ixy="${0.00155092*density}" ixz="${-0.00000053*density}"
+	  iyy="${0.00131780*density}" iyz="${0.00000195*density}"
+	  izz="${0.00607489*density}"/>
     </inertial>
     <visual>
@@ -266,11 +267,11 @@
     <inertial>
       <origin
-        xyz="-0.0159722248323729 -0.0365908819941969 2.28756223330485E-06"
-        rpy="0 0 0" />
-      <mass value="0.05"/>
-      <inertia
-	  ixx="0.001" ixy="0.0" ixz="0.0"
-	  iyy="0.001" iyz="0.0"
-	  izz="0.001"/>
+        xyz="-0.0159154 -0.0365660 0.0000004"
+        rpy="0 0 0" />
+      <mass value="${0.808399*density}"/>
+      <inertia
+	  ixx="${0.00194399*density}" ixy="${0.00047414*density}" ixz="${0.00000001*density}"
+	  iyy="${0.00113245*density}" iyz="${-0.00000012*density}"
+	  izz="${0.00246661*density}"/>
     </inertial>
     <visual>
@@ -317,11 +318,11 @@
     <inertial>
       <origin
-        xyz="-0.0390479629436857 0.693839823742315 0.000123076547971226"
-        rpy="0 0 0" />
-      <mass value="0.05"/>
-      <inertia
-	  ixx="0.001" ixy="0.0" ixz="0.0"
-	  iyy="0.001" iyz="0.0"
-	  izz="0.001"/>
+        xyz="-0.0009237 -0.042691 -0.0003367"
+        rpy="0 0 0" />
+      <mass value="${0.147312*density}"/>
+      <inertia
+	  ixx="${0.00045468*density}" ixy="${-0.00006666*density}" ixz="${-0.00000289*density}"
+	  iyy="${0.00019592*density}" iyz="${-0.00002477*density}"
+	  izz="${0.00045557*density}"/>
     </inertial>
     <visual>
