Commit message: update elfin3.urdf.xacro and elfin10.urdf.xacro for color

File: elfin_description/urdf/elfin10.urdf.xacro (robot description, xacro)
@@ -50,8 +50,5 @@
       </geometry>
       <material
-        name="">
-        <color
-          rgba="0.792156862745098 0.819607843137255 0.925490196078431 1" />
-      </material>
+        name="metal_white"/>
     </visual>
     <collision>
@@ -90,8 +87,5 @@
       </geometry>
       <material
-        name="">
-        <color
-          rgba="1 1 1 1" />
-      </material>
+        name="metal"/>
     </visual>
     <collision>
@@ -148,8 +142,5 @@
       </geometry>
       <material
-        name="">
-        <color
-          rgba="0.501960784313725 0.501960784313725 0.501960784313725 1" />
-      </material>
+        name="metal_grey"/>
     </visual>
     <collision>
@@ -206,8 +197,5 @@
       </geometry>
       <material
-        name="">
-        <color
-          rgba="1 1 1 1" />
-      </material>
+        name="metal"/>
     </visual>
     <collision>
@@ -264,8 +252,5 @@
       </geometry>
       <material
-        name="">
-        <color
-          rgba="0.501960784313725 0.501960784313725 0.501960784313725 1" />
-      </material>
+        name="metal_grey"/>
     </visual>
     <collision>
@@ -322,8 +307,5 @@
       </geometry>
       <material
-        name="">
-        <color
-          rgba="1 1 1 1" />
-      </material>
+        name="metal"/>
     </visual>
     <collision>
@@ -380,8 +362,5 @@
       </geometry>
       <material
-        name="">
-        <color
-          rgba="0.792156862745098 0.819607843137255 0.929411764705882 1" />
-      </material>
+        name="metal_white"/>
     </visual>
     <collision>

File: elfin_description/urdf/elfin3.urdf.xacro (robot description, xacro)
@@ -50,8 +50,5 @@
       </geometry>
       <material
-        name="">
-        <color
-          rgba="0.686274509803922 0.686274509803922 0.686274509803922 1" />
-      </material>
+        name="metal_white"/>
     </visual>
     <collision>
@@ -90,8 +87,5 @@
       </geometry>
       <material
-        name="">
-        <color
-          rgba="0.768627450980392 0.749019607843137 0.729411764705882 1" />
-      </material>
+        name="metal"/>
     </visual>
     <collision>
@@ -148,8 +142,5 @@
       </geometry>
       <material
-        name="">
-        <color
-          rgba="0.501960784313725 0.501960784313725 0.501960784313725 1" />
-      </material>
+        name="metal_grey"/>
     </visual>
     <collision>
@@ -206,8 +197,5 @@
       </geometry>
       <material
-        name="">
-        <color
-          rgba="1 1 1 1" />
-      </material>
+        name="metal"/>
     </visual>
     <collision>
@@ -264,8 +252,5 @@
       </geometry>
       <material
-        name="">
-        <color
-          rgba="0.501960784313725 0.501960784313725 0.501960784313725 1" />
-      </material>
+        name="metal_grey"/>
     </visual>
     <collision>
@@ -322,8 +307,5 @@
       </geometry>
       <material
-        name="">
-        <color
-          rgba="0.768627450980392 0.749019607843137 0.729411764705882 1" />
-      </material>
+        name="metal"/>
     </visual>
     <collision>
@@ -380,8 +362,5 @@
       </geometry>
       <material
-        name="">
-        <color
-          rgba="0.866666666666667 0.866666666666667 0.890196078431373 1" />
-      </material>
+        name="metal_white"/>
     </visual>
     <collision>

Commit message: update inertia of robot models

File: elfin_description/urdf/elfin10.urdf.xacro (robot description, xacro)
@@ -31,13 +31,9 @@
         xyz="0.000308020598430213 0.027286204143835 -0.00272949562920981"
         rpy="0 0 0" />
-      <mass
-        value="0.885375178384734" />
-      <inertia
-        ixx="0.00286318889286201"
-        ixy="3.45365039921659E-06"
-        ixz="-1.62402262526516E-05"
-        iyy="0.00535727192521691"
-        iyz="-2.78342487667673E-05"
-        izz="0.00303602788914978" />
+      <mass value="0.05"/>
+      <inertia
+	  ixx="0.001" ixy="0.0" ixz="0.0"
+	  iyy="0.001" iyz="0.0"
+	  izz="0.001"/>
     </inertial>
     <visual>
@@ -68,13 +64,9 @@
         xyz="-0.025606009350082 0.195630799437867 1.98466916955487E-05"
         rpy="0 0 0" />
-      <mass
-        value="5.0663557884435" />
-      <inertia
-        ixx="0.0400804338380401"
-        ixy="0.00849162788349833"
-        ixz="-5.6134782300454E-06"
-        iyy="0.0212587213618438"
-        iyz="-2.4294887610495E-06"
-        izz="0.0457568717782572" />
+      <mass value="0.05"/>
+      <inertia
+	  ixx="0.001" ixy="0.0" ixz="0.0"
+	  iyy="0.001" iyz="0.0"
+	  izz="0.001"/>
     </inertial>
     <visual>
@@ -123,13 +115,9 @@
         xyz="-0.059127689307098 0.209937989447816 7.56723981552217E-06"
         rpy="0 0 0" />
-      <mass
-        value="1.67188352649654" />
-      <inertia
-        ixx="0.0525625660873116"
-        ixy="-0.00220862698349637"
-        ixz="-6.2414828525538E-07"
-        iyy="0.00437200496167382"
-        iyz="-9.38433431531435E-06"
-        izz="0.0512001113698696" />
+      <mass value="0.05"/>
+      <inertia
+	  ixx="0.001" ixy="0.0" ixz="0.0"
+	  iyy="0.001" iyz="0.0"
+	  izz="0.001"/>
     </inertial>
     <visual>
@@ -178,13 +166,9 @@
         xyz="0.0625123989669429 -0.052176807477553 2.64760976133438E-05"
         rpy="0 0 0" />
-      <mass
-        value="2.52856215211273" />
-      <inertia
-        ixx="0.012667847540505"
-        ixy="0.00290607544164991"
-        ixz="-1.47525213406371E-06"
-        iyy="0.00711624913901914"
-        iyz="-2.69674594651337E-06"
-        izz="0.0150236128176268" />
+      <mass value="0.05"/>
+      <inertia
+	  ixx="0.001" ixy="0.0" ixz="0.0"
+	  iyy="0.001" iyz="0.0"
+	  izz="0.001"/>
     </inertial>
     <visual>
@@ -233,13 +217,9 @@
         xyz="-0.0655191412736019 0.17921070701944 1.42681979805022E-05"
         rpy="0 0 0" />
-      <mass
-        value="0.774714242593802" />
-      <inertia
-        ixx="0.0125887055785559"
-        ixy="0.00311217340021864"
-        ixz="4.28455933012487E-08"
-        iyy="0.00273673242411354"
-        iyz="6.42522589973016E-07"
-        izz="0.0136908740275145" />
+      <mass value="0.05"/>
+      <inertia
+	  ixx="0.001" ixy="0.0" ixz="0.0"
+	  iyy="0.001" iyz="0.0"
+	  izz="0.001"/>
     </inertial>
     <visual>
@@ -288,13 +268,9 @@
         xyz="-0.0175084997767369 -0.0377654900394784 -7.04779685984352E-06"
         rpy="0 0 0" />
-      <mass
-        value="1.07922052439642" />
-      <inertia
-        ixx="0.00298738623352246"
-        ixy="0.000725824515360465"
-        ixz="4.96155482882277E-07"
-        iyy="0.00183400932518434"
-        iyz="-2.66412614052824E-07"
-        izz="0.00375395523653828" />
+      <mass value="0.05"/>
+      <inertia
+	  ixx="0.001" ixy="0.0" ixz="0.0"
+	  iyy="0.001" iyz="0.0"
+	  izz="0.001"/>
     </inertial>
     <visual>
@@ -343,13 +319,9 @@
         xyz="-0.0412046461038743 -0.870077360796272 -0.000195877685084774"
         rpy="0 0 0" />
-      <mass
-        value="12.0061109281425" />
-      <inertia
-        ixx="1.92519773999221"
-        ixy="0.0176915240535981"
-        ixz="7.99693876355251E-05"
-        iyy="0.0649687530706708"
-        iyz="-0.00114805616509498"
-        izz="1.9561905498035" />
+      <mass value="0.05"/>
+      <inertia
+	  ixx="0.001" ixy="0.0" ixz="0.0"
+	  iyy="0.001" iyz="0.0"
+	  izz="0.001"/>
     </inertial>
     <visual>

File: elfin_description/urdf/elfin3.urdf.xacro (robot description, xacro)
@@ -31,13 +31,9 @@
         xyz="-0.0319402056221453 0.427120668618383 -5.39351164605318E-06"
         rpy="0 0 0" />
-      <mass
-        value="4.3052612459755" />
-      <inertia
-        ixx="0.291480854811486"
-        ixy="-0.00222433961096429"
-        ixz="-2.01923964457691E-06"
-        iyy="0.0113685309214344"
-        iyz="-3.62155285906403E-06"
-        izz="0.298007263296196" />
+      <mass value="0.05"/>
+      <inertia
+	  ixx="0.001" ixy="0.0" ixz="0.0"
+	  iyy="0.001" iyz="0.0"
+	  izz="0.001"/>
     </inertial>
     <visual>
@@ -68,13 +64,9 @@
         xyz="-0.0192918165822649 0.120142940373248 -9.33059379656128E-06"
         rpy="0 0 0" />
-      <mass
-        value="1.52637984956046" />
-      <inertia
-        ixx="0.00527544044696735"
-        ixy="0.00123465778378514"
-        ixz="-6.71312813911233E-07"
-        iyy="0.00317642212936588"
-        iyz="-3.23660070050034E-07"
-        izz="0.00651212770034193" />
+      <mass value="0.05"/>
+      <inertia
+	  ixx="0.001" ixy="0.0" ixz="0.0"
+	  iyy="0.001" iyz="0.0"
+	  izz="0.001"/>
     </inertial>
     <visual>
@@ -123,13 +115,9 @@
         xyz="-0.036466516774824 0.121897297057332 -2.81161718183357E-05"
         rpy="0 0 0" />
-      <mass
-        value="0.519454683951505" />
-      <inertia
-        ixx="0.00565995615696724"
-        ixy="-0.000264286704227211"
-        ixz="9.00238413174917E-08"
-        iyy="0.000537503501646015"
-        iyz="2.30075042384658E-06"
-        izz="0.00546582402574428" />
+      <mass value="0.05"/>
+      <inertia
+	  ixx="0.001" ixy="0.0" ixz="0.0"
+	  iyy="0.001" iyz="0.0"
+	  izz="0.001"/>
     </inertial>
     <visual>
@@ -178,13 +166,9 @@
         xyz="0.0512991448419209 -0.0377654897323815 -7.04730066125333E-06"
         rpy="0 0 0" />
-      <mass
-        value="1.07922053966635" />
-      <inertia
-        ixx="0.00298738624023049"
-        ixy="0.000725824493179576"
-        ixz="4.96115488717236E-07"
-        iyy="0.00183400941739145"
-        iyz="-2.66433909735348E-07"
-        izz="0.00375395532323906" />
+      <mass value="0.05"/>
+      <inertia
+	  ixx="0.001" ixy="0.0" ixz="0.0"
+	  iyy="0.001" iyz="0.0"
+	  izz="0.001"/>
     </inertial>
     <visual>
@@ -233,13 +217,9 @@
         xyz="-0.0583601900884385 0.100119219162888 -3.33183498268088E-07"
         rpy="0 0 0" />
-      <mass
-        value="0.369677539276185" />
-      <inertia
-        ixx="0.00237292271100579"
-        ixy="0.000824081879058636"
-        ixz="-8.45848544546041E-09"
-        iyy="0.000956009074525509"
-        iyz="-3.93294162811061E-09"
-        izz="0.00283923133217817" />
+      <mass value="0.05"/>
+      <inertia
+	  ixx="0.001" ixy="0.0" ixz="0.0"
+	  iyy="0.001" iyz="0.0"
+	  izz="0.001"/>
     </inertial>
     <visual>
@@ -288,13 +268,9 @@
         xyz="-0.0159268625326372 -0.0365461558991834 2.29158666616884E-06"
         rpy="0 0 0" />
-      <mass
-        value="0.81052865799498" />
-      <inertia
-        ixx="0.00195203104787827"
-        ixy="0.000475249185078403"
-        ixz="-4.08714933153791E-08"
-        iyy="0.0011361781195507"
-        iyz="1.7320616235908E-08"
-        izz="0.00247459893149932" />
+      <mass value="0.05"/>
+      <inertia
+	  ixx="0.001" ixy="0.0" ixz="0.0"
+	  iyy="0.001" iyz="0.0"
+	  izz="0.001"/>
     </inertial>
     <visual>
@@ -343,13 +319,9 @@
         xyz="0.0219175619250529 0.461879324434722 -0.0232335370431645"
         rpy="0 0 0" />
-      <mass
-        value="4.3052612459755" />
-      <inertia
-        ixx="0.294935032119192"
-        ixy="-0.0015239945221609"
-        ixz="0.0032576119002927"
-        iyy="0.0113685309214282"
-        iyz="0.00162022853851308"
-        izz="0.294553085988403" />
+      <mass value="0.05"/>
+      <inertia
+	  ixx="0.001" ixy="0.0" ixz="0.0"
+	  iyy="0.001" iyz="0.0"
+	  izz="0.001"/>
     </inertial>
     <visual>

File: elfin_description/urdf/elfin5.urdf.xacro (robot description, xacro)
@@ -31,13 +31,9 @@
         xyz="0.000220821977982989 0.0255290818849933 -0.00134044659901771"
         rpy="0 0 0" />
-      <mass
-        value="0.687962637332097" />
-      <inertia
-        ixx="0.00130306123187478"
-        ixy="1.96861257772613E-06"
-        ixz="-5.74929479012133E-06"
-        iyy="0.00228919563106407"
-        iyz="-1.11186982812778E-05"
-        izz="0.00134151625913869" />
+      <mass value="0.05"/>
+      <inertia
+	  ixx="0.001" ixy="0.0" ixz="0.0"
+	  iyy="0.001" iyz="0.0"
+	  izz="0.001"/>
     </inertial>
     <visual>
@@ -68,13 +64,9 @@
         xyz="-0.0218141046310325 0.138891728726282 1.31241816829816E-05"
         rpy="0 0 0" />
-      <mass
-        value="2.58573759197982" />
-      <inertia
-        ixx="0.0130674681894722"
-        ixy="0.0028998968693497"
-        ixz="-1.29833068203639E-06"
-        iyy="0.00725121580985117"
-        iyz="-1.21845402845366E-06"
-        izz="0.015419294302391" />
+      <mass value="0.05"/>
+      <inertia
+	  ixx="0.001" ixy="0.0" ixz="0.0"
+	  iyy="0.001" iyz="0.0"
+	  izz="0.001"/>
     </inertial>
     <visual>
@@ -123,13 +115,9 @@
         xyz="-0.0524295669840444 0.158140141659462 -1.74919824000372E-06"
         rpy="0 0 0" />
-      <mass
-        value="1.21317989660263" />
-      <inertia
-        ixx="0.0298439491889078"
-        ixy="-0.00126866698999722"
-        ixz="-8.69205913477971E-08"
-        iyy="0.00168968241043964"
-        iyz="-1.17248720067113E-06"
-        izz="0.0295226476065225" />
+      <mass value="0.05"/>
+      <inertia
+	  ixx="0.001" ixy="0.0" ixz="0.0"
+	  iyy="0.001" iyz="0.0"
+	  izz="0.001"/>
     </inertial>
     <visual>
@@ -178,13 +166,9 @@
         xyz="0.0586561082766824 -0.0414791884757505 -9.80549635387022E-06"
         rpy="0 0 0" />
-      <mass
-        value="1.53247101114637" />
-      <inertia
-        ixx="0.00531714403008397"
-        ixy="0.00125082388816858"
-        ixz="-6.89885730487444E-07"
-        iyy="0.00320121076269661"
-        iyz="-3.61767642380346E-07"
-        izz="0.00657309788563969" />
+      <mass value="0.05"/>
+      <inertia
+	  ixx="0.001" ixy="0.0" ixz="0.0"
+	  iyy="0.001" iyz="0.0"
+	  izz="0.001"/>
     </inertial>
     <visual>
@@ -233,13 +217,9 @@
         xyz="-0.0589525602581192 0.143654952750886 -4.64578965075454E-05"
         rpy="0 0 0" />
-      <mass
-        value="0.475173202131869" />
-      <inertia
-        ixx="0.00542665349810737"
-        ixy="0.00154907507395157"
-        ixz="-8.54435811246923E-07"
-        iyy="0.00132021432350494"
-        iyz="2.50752623988858E-06"
-        izz="0.00607595548033839" />
+      <mass value="0.05"/>
+      <inertia
+	  ixx="0.001" ixy="0.0" ixz="0.0"
+	  iyy="0.001" iyz="0.0"
+	  izz="0.001"/>
     </inertial>
     <visual>
@@ -288,13 +268,9 @@
         xyz="-0.0159722248323729 -0.0365908819941969 2.28756223330485E-06"
         rpy="0 0 0" />
-      <mass
-        value="0.811929382825872" />
-      <inertia
-        ixx="0.00195893851194632"
-        ixy="0.000477990571584107"
-        ixz="-4.77934949619082E-08"
-        iyy="0.0011401479695366"
-        iyz="5.38748772660695E-09"
-        izz="0.0024848311864596" />
+      <mass value="0.05"/>
+      <inertia
+	  ixx="0.001" ixy="0.0" ixz="0.0"
+	  iyy="0.001" iyz="0.0"
+	  izz="0.001"/>
     </inertial>
     <visual>
@@ -343,13 +319,9 @@
         xyz="-0.0390479629436857 0.693839823742315 0.000123076547971226"
         rpy="0 0 0" />
-      <mass
-        value="7.30645413254167" />
-      <inertia
-        ixx="0.822951027515021"
-        ixy="-0.00419851067785738"
-        ixz="-2.7490901915861E-05"
-        iyy="0.0300791191703889"
-        iyz="-0.000370584165009564"
-        izz="0.840636353527808" />
+      <mass value="0.05"/>
+      <inertia
+	  ixx="0.001" ixy="0.0" ixz="0.0"
+	  iyy="0.001" iyz="0.0"
+	  izz="0.001"/>
     </inertial>
     <visual>
