Commit message: correct the inertial parameters in urdf models

File: elfin_description/urdf/elfin10.urdf.xacro (robot description, xacro)
@@ -5,4 +5,5 @@
   <xacro:include filename="$(find elfin_description)/urdf/elfin_transmission.xacro" />
   <xacro:property name="PI" value="3.1415926535897931"/>
+  <xacro:property name="density" value="3.09"/>
   <link name="world"/>
   <joint name="world_base" type="fixed">
@@ -29,11 +30,11 @@
     <inertial>
       <origin
-        xyz="0.000308020598430213 0.027286204143835 -0.00272949562920981"
-        rpy="0 0 0" />
-      <mass value="0.05"/>
-      <inertia
-	  ixx="0.001" ixy="0.0" ixz="0.0"
-	  iyy="0.001" iyz="0.0"
-	  izz="0.001"/>
+        xyz="0.00029790659221 0.00271788312044 0.0274159041935"
+        rpy="0 0 0"/>
+      <mass value="${0.890680700037*density}"/>
+      <inertia
+      ixx="${0.00287631*density}" ixy="${1.617e-05*density}" ixz="${3.38e-06*density}"
+      iyy="${0.00304792*density}" iyz="${2.79e-05*density}"
+      izz="${0.00537429*density}"/>
     </inertial>
     <visual>
@@ -62,11 +63,11 @@
     <inertial>
       <origin
-        xyz="-0.025606009350082 0.195630799437867 1.98466916955487E-05"
-        rpy="0 0 0" />
-      <mass value="0.05"/>
-      <inertia
-	  ixx="0.001" ixy="0.0" ixz="0.0"
-	  iyy="0.001" iyz="0.0"
-	  izz="0.001"/>
+        xyz="-0.0255519176997 0.195603533565 1.68999482169e-05"
+        rpy="0 0 0"/>
+      <mass value="${5.04797690664*density}"/>
+      <inertia
+      ixx="${0.03982126*density}" ixy="${0.00844769*density}" ixz="${-4.29e-06*density}"
+      iyy="${0.02114179*density}" iyz="${-2.23e-06*density}"
+      izz="${0.04547525*density}"/>
     </inertial>
     <visual>
@@ -113,11 +114,11 @@
     <inertial>
       <origin
-        xyz="-0.059127689307098 0.209937989447816 7.56723981552217E-06"
-        rpy="0 0 0" />
-      <mass value="0.05"/>
-      <inertia
-	  ixx="0.001" ixy="0.0" ixz="0.0"
-	  iyy="0.001" iyz="0.0"
-	  izz="0.001"/>
+        xyz="-0.0589642426226 0.20968040657 -5.33587812464e-06"
+        rpy="0 0 0"/>
+      <mass value="${1.66596877354*density}"/>
+      <inertia
+      ixx="${0.052412*density}" ixy="${-0.00219612*density}" ixz="${-1.07e-06*density}"
+      iyy="${0.00434323*density}" iyz="${-1.255e-05*density}"
+      izz="${0.05107023*density}"/>
     </inertial>
     <visual>
@@ -164,11 +165,11 @@
     <inertial>
       <origin
-        xyz="0.0625123989669429 -0.052176807477553 2.64760976133438E-05"
-        rpy="0 0 0" />
-      <mass value="0.05"/>
-      <inertia
-	  ixx="0.001" ixy="0.0" ixz="0.0"
-	  iyy="0.001" iyz="0.0"
-	  izz="0.001"/>
+        xyz="0.0625690665762 -0.0521846187635 2.58799082907e-05"
+        rpy="0 0 0"/>
+      <mass value="${2.51986584925*density}"/>
+      <inertia
+      ixx="${0.01259396*density}" ixy="${0.00288795*density}" ixz="${-1.16e-06*density}"
+      iyy="${0.00707893*density}" iyz="${-2.15e-06*density}"
+      izz="${0.01493778*density}"/>
     </inertial>
     <visual>
@@ -215,11 +216,11 @@
     <inertial>
       <origin
-        xyz="-0.0655191412736019 0.17921070701944 1.42681979805022E-05"
-        rpy="0 0 0" />
-      <mass value="0.05"/>
-      <inertia
-	  ixx="0.001" ixy="0.0" ixz="0.0"
-	  iyy="0.001" iyz="0.0"
-	  izz="0.001"/>
+        xyz="-0.0653325107739 0.17924183252 -8.22522528991e-06"
+        rpy="0 0 0"/>
+      <mass value="${0.773882513506*density}"/>
+      <inertia
+      ixx="${0.01260891*density}" ixy="${0.00311563*density}" ixz="${5.8e-07*density}"
+      iyy="${0.00272662*density}" iyz="${-1.47e-06*density}"
+      izz="${0.01371082*density}"/>
     </inertial>
     <visual>
@@ -266,11 +267,11 @@
     <inertial>
       <origin
-        xyz="-0.0175084997767369 -0.0377654900394784 -7.04779685984352E-06"
-        rpy="0 0 0" />
-      <mass value="0.05"/>
-      <inertia
-	  ixx="0.001" ixy="0.0" ixz="0.0"
-	  iyy="0.001" iyz="0.0"
-	  izz="0.001"/>
+        xyz="-0.0174451255278 -0.0377419055039 -1.41483594707e-05"
+        rpy="0 0 0"/>
+      <mass value="${1.07514483832*density}"/>
+      <inertia
+      ixx="${0.00296619*density}" ixy="${0.00072021*density}" ixz="${7.3e-07*density}"
+      iyy="${0.00182263*density}" iyz="${-3.7e-07*density}"
+      izz="${0.00372855*density}"/>
     </inertial>
     <visual>
@@ -317,11 +318,11 @@
     <inertial>
       <origin
-        xyz="-0.0412046461038743 -0.870077360796272 -0.000195877685084774"
-        rpy="0 0 0" />
-      <mass value="0.05"/>
-      <inertia
-	  ixx="0.001" ixy="0.0" ixz="0.0"
-	  iyy="0.001" iyz="0.0"
-	  izz="0.001"/>
+        xyz="0.00115745849085 0.0594966864835 0.000222299836983"
+        rpy="0 0 0"/>
+      <mass value="${0.184390264995*density}"/>
+      <inertia
+      ixx="${0.00077254*density}" ixy="${-3.97e-06*density}" ixz="${-1.29e-06*density}"
+      iyy="${0.0002179*density}" iyz="${-8.1e-07*density}"
+      izz="${0.00078406*density}"/>
     </inertial>
     <visual>

File: elfin_description/urdf/elfin3.urdf.xacro (robot description, xacro)
@@ -5,4 +5,5 @@
   <xacro:include filename="$(find elfin_description)/urdf/elfin_transmission.xacro" />
   <xacro:property name="PI" value="3.1415926535897931"/>
+  <xacro:property name="density" value="3.09"/>
   <link name="world"/>
   <joint name="world_base" type="fixed">
@@ -29,11 +30,11 @@
     <inertial>
       <origin
-        xyz="-0.0319402056221453 0.427120668618383 -5.39351164605318E-06"
-        rpy="0 0 0" />
-      <mass value="0.05"/>
-      <inertia
-	  ixx="0.001" ixy="0.0" ixz="0.0"
-	  iyy="0.001" iyz="0.0"
-	  izz="0.001"/>
+        xyz="0.000476057496448 -0.00609847721085 0.0271227961552"
+        rpy="0 0 0"/>
+      <mass value="${0.432503561632*density}"/>
+      <inertia
+      ixx="${0.00107966*density}" ixy="${6.43e-06*density}" ixz="${1.97e-06*density}"
+      iyy="${0.00089216*density}" iyz="${-1.269e-05*density}"
+      izz="${0.00174712*density}"/>
     </inertial>
     <visual>
@@ -62,11 +63,11 @@
     <inertial>
       <origin
-        xyz="-0.0192918165822649 0.120142940373248 -9.33059379656128E-06"
-        rpy="0 0 0" />
-      <mass value="0.05"/>
-      <inertia
-	  ixx="0.001" ixy="0.0" ixz="0.0"
-	  iyy="0.001" iyz="0.0"
-	  izz="0.001"/>
+        xyz="-0.0192425632808 0.120157543892 -2.05350524914e-05"
+        rpy="0 0 0"/>
+      <mass value="${1.52001312557*density}"/>
+      <inertia
+      ixx="${0.00523815*density}" ixy="${0.00122593*density}" ixz="${-1.6e-07*density}"
+      iyy="${0.00315471*density}" iyz="${-6.4e-07*density}"
+      izz="${0.00646649*density}"/>
     </inertial>
     <visual>
@@ -113,11 +114,11 @@
     <inertial>
       <origin
-        xyz="-0.036466516774824 0.121897297057332 -2.81161718183357E-05"
-        rpy="0 0 0" />
-      <mass value="0.05"/>
-      <inertia
-	  ixx="0.001" ixy="0.0" ixz="0.0"
-	  iyy="0.001" iyz="0.0"
-	  izz="0.001"/>
+        xyz="-0.0363359816546 0.121774838175 -3.84046105722e-05"
+        rpy="0 0 0"/>
+      <mass value="${0.519672255247*density}"/>
+      <inertia
+      ixx="${0.00564813*density}" ixy="${-0.00026473*density}" ixz="${0.0*density}"
+      iyy="${0.00053594*density}" iyz="${1.29e-06*density}"
+      izz="${0.00545618*density}"/>
     </inertial>
     <visual>
@@ -164,11 +165,11 @@
     <inertial>
       <origin
-        xyz="0.0512991448419209 -0.0377654897323815 -7.04730066125333E-06"
-        rpy="0 0 0" />
-      <mass value="0.05"/>
-      <inertia
-	  ixx="0.001" ixy="0.0" ixz="0.0"
-	  iyy="0.001" iyz="0.0"
-	  izz="0.001"/>
+        xyz="0.0513625008301 -0.0377418700977 -1.41484011876e-05"
+        rpy="0 0 0"/>
+      <mass value="${1.07514585114*density}"/>
+      <inertia
+      ixx="${0.00296619*density}" ixy="${0.00072021*density}" ixz="${7.3e-07*density}"
+      iyy="${0.00182263*density}" iyz="${-3.7e-07*density}"
+      izz="${0.00372855*density}"/>
     </inertial>
     <visual>
@@ -215,11 +216,11 @@
     <inertial>
       <origin
-        xyz="-0.0583601900884385 0.100119219162888 -3.33183498268088E-07"
-        rpy="0 0 0" />
-      <mass value="0.05"/>
-      <inertia
-	  ixx="0.001" ixy="0.0" ixz="0.0"
-	  iyy="0.001" iyz="0.0"
-	  izz="0.001"/>
+        xyz="-0.0580853772834 0.10002233137 -3.45203877103e-06"
+        rpy="0 0 0"/>
+      <mass value="${0.37026646381*density}"/>
+      <inertia
+      ixx="${0.00238279*density}" ixy="${0.00082955*density}" ixz="${1.1e-07*density}"
+      iyy="${0.00095758*density}" iyz="${-3.2e-07*density}"
+      izz="${0.00285161*density}"/>
     </inertial>
     <visual>
@@ -266,11 +267,11 @@
     <inertial>
       <origin
-        xyz="-0.0159268625326372 -0.0365461558991834 2.29158666616884E-06"
-        rpy="0 0 0" />
-      <mass value="0.05"/>
-      <inertia
-	  ixx="0.001" ixy="0.0" ixz="0.0"
-	  iyy="0.001" iyz="0.0"
-	  izz="0.001"/>
+        xyz="-0.0158710385319 -0.0365214098995 4.94388107361e-07"
+        rpy="0 0 0"/>
+      <mass value="${0.807027243448*density}"/>
+      <inertia
+      ixx="${0.00193719*density}" ixy="${0.00047145*density}" ixz="${2e-08*density}"
+      iyy="${0.00112857*density}" iyz="${-1.1e-07*density}"
+      izz="${0.00245655*density}"/>
     </inertial>
     <visual>
@@ -317,11 +318,11 @@
     <inertial>
       <origin
-        xyz="0.0219175619250529 0.461879324434722 -0.0232335370431645"
-        rpy="0 0 0" />
-      <mass value="0.05"/>
-      <inertia
-	  ixx="0.001" ixy="0.0" ixz="0.0"
-	  iyy="0.001" iyz="0.0"
-	  izz="0.001"/>
+        xyz="-0.000923639476392 -0.0528295663466 -0.000336667608557"
+        rpy="0 0 0"/>
+      <mass value="${0.147312568674*density}"/>
+      <inertia
+      ixx="${0.00057253*density}" ixy="${-2.66e-06*density}" ixz="${-2.89e-06*density}"
+      iyy="${0.00019592*density}" iyz="${-1.2e-06*density}"
+      izz="${0.00057342*density}"/>
     </inertial>
     <visual>

File: elfin_description/urdf/elfin5.urdf.xacro (robot description, xacro)
@@ -34,7 +34,7 @@
       <mass value="${0.690521*density}"/>
       <inertia
-	  ixx="${0.00130611*density}" ixy="${0.0000568*density}" ixz="${0.00000189*density}"
-	  iyy="${0.00134467*density}" iyz="${0.00001095*density}"
-	  izz="${0.00229139*density}"/>
+      ixx="${0.00130611*density}" ixy="${0.0000568*density}" ixz="${0.00000189*density}"
+      iyy="${0.00134467*density}" iyz="${0.00001095*density}"
+      izz="${0.00229139*density}"/>
     </inertial>
     <visual>
@@ -67,7 +67,7 @@
       <mass value="${2.576772*density}"/>
       <inertia
-	  ixx="${0.01298966*density}" ixy="${0.00287966*density}" ixz="${-0.000001*density}"
-	  iyy="${0.00721115*density}" iyz="${-0.00000052*density}"
-	  izz="${0.01532713*density}"/>
+      ixx="${0.01298966*density}" ixy="${0.00287966*density}" ixz="${-0.000001*density}"
+      iyy="${0.00721115*density}" iyz="${-0.00000052*density}"
+      izz="${0.01532713*density}"/>
     </inertial>
     <visual>
@@ -118,7 +118,7 @@
       <mass value="${1.208607*density}"/>
       <inertia
-	  ixx="${0.02975970*density}" ixy="${-0.00126441*density}" ixz="${-0.00000024*density}"
-	  iyy="${0.00168156*density}" iyz="${-0.0000021*density}"
-	  izz="${0.02944694*density}"/>
+      ixx="${0.02975970*density}" ixy="${-0.00126441*density}" ixz="${-0.00000024*density}"
+      iyy="${0.00168156*density}" iyz="${-0.0000021*density}"
+      izz="${0.02944694*density}"/>
     </inertial>
     <visual>
@@ -169,7 +169,7 @@
       <mass value="${1.525883*density}"/>
       <inertia
-	  ixx="${0.00527835*density}" ixy="${0.00124150*density}" ixz="${-0.00000018*density}"
-	  iyy="${0.00317861*density}" iyz="${-0.00000067*density}"
-	  izz="${0.00652527*density}"/>
+      ixx="${0.00527835*density}" ixy="${0.00124150*density}" ixz="${-0.00000018*density}"
+      iyy="${0.00317861*density}" iyz="${-0.00000067*density}"
+      izz="${0.00652527*density}"/>
     </inertial>
     <visual>
@@ -220,7 +220,7 @@
       <mass value="${0.475026*density}"/>
       <inertia
-	  ixx="${0.00542441*density}" ixy="${0.00155092*density}" ixz="${-0.00000053*density}"
-	  iyy="${0.00131780*density}" iyz="${0.00000195*density}"
-	  izz="${0.00607489*density}"/>
+      ixx="${0.00542441*density}" ixy="${0.00155092*density}" ixz="${-0.00000053*density}"
+      iyy="${0.00131780*density}" iyz="${0.00000195*density}"
+      izz="${0.00607489*density}"/>
     </inertial>
     <visual>
@@ -271,7 +271,7 @@
       <mass value="${0.808399*density}"/>
       <inertia
-	  ixx="${0.00194399*density}" ixy="${0.00047414*density}" ixz="${0.00000001*density}"
-	  iyy="${0.00113245*density}" iyz="${-0.00000012*density}"
-	  izz="${0.00246661*density}"/>
+      ixx="${0.00194399*density}" ixy="${0.00047414*density}" ixz="${0.00000001*density}"
+      iyy="${0.00113245*density}" iyz="${-0.00000012*density}"
+      izz="${0.00246661*density}"/>
     </inertial>
     <visual>
@@ -322,7 +322,7 @@
       <mass value="${0.147312*density}"/>
       <inertia
-	  ixx="${0.00045468*density}" ixy="${-0.00006666*density}" ixz="${-0.00000289*density}"
-	  iyy="${0.00019592*density}" iyz="${-0.00002477*density}"
-	  izz="${0.00045557*density}"/>
+      ixx="${0.00045468*density}" ixy="${-0.000005401*density}" ixz="${-0.00000289*density}"
+      iyy="${0.00019592*density}" iyz="${-0.000002430*density}"
+      izz="${0.00045557*density}"/>
     </inertial>
     <visual>

Commit message: update urdf models

File: elfin_description/urdf/elfin10.urdf.xacro (robot description, xacro)
@@ -322,7 +322,7 @@
       <mass value="${0.184390264995*density}"/>
       <inertia
-      ixx="${0.00077254*density}" ixy="${-3.97e-06*density}" ixz="${-1.29e-06*density}"
-      iyy="${0.0002179*density}" iyz="${-8.1e-07*density}"
-      izz="${0.00078406*density}"/>
+      ixx="${0.00018992*density}" ixy="${4.57e-06*density}" ixz="${-1.29e-06*density}"
+      iyy="${0.0002179*density}" iyz="${8.3e-07*density}"
+      izz="${0.00020144*density}"/>
     </inertial>
     <visual>

File: elfin_description/urdf/elfin3.urdf.xacro (robot description, xacro)
@@ -318,11 +318,11 @@
     <inertial>
       <origin
-        xyz="-0.000923639476392 -0.0528295663466 -0.000336667608557"
-        rpy="0 0 0"/>
-      <mass value="${0.147312568674*density}"/>
-      <inertia
-      ixx="${0.00057253*density}" ixy="${-2.66e-06*density}" ixz="${-2.89e-06*density}"
-      iyy="${0.00019592*density}" iyz="${-1.2e-06*density}"
-      izz="${0.00057342*density}"/>
+        xyz="-0.0009237 -0.042691 -0.0003367"
+        rpy="0 0 0" />
+      <mass value="${0.147312*density}"/>
+      <inertia
+      ixx="${0.00019407*density}" ixy="${1.4e-06*density}" ixz="${-2.89e-06*density}"
+      iyy="${0.00019592*density}" iyz="${5e-08*density}"
+      izz="${0.00019496*density}"/>
     </inertial>
     <visual>

File: elfin_description/urdf/elfin5.urdf.xacro (robot description, xacro)
@@ -322,7 +322,7 @@
       <mass value="${0.147312*density}"/>
       <inertia
-      ixx="${0.00045468*density}" ixy="${-0.000005401*density}" ixz="${-0.00000289*density}"
-      iyy="${0.00019592*density}" iyz="${-0.000002430*density}"
-      izz="${0.00045557*density}"/>
+      ixx="${0.00019407*density}" ixy="${1.4e-06*density}" ixz="${-2.89e-06*density}"
+      iyy="${0.00019592*density}" iyz="${5e-08*density}"
+      izz="${0.00019496*density}"/>
     </inertial>
     <visual>
