Commit message: update model and urdf
update elfin3/elfin5/elfin10/module_14 model and urdf, add module_25

File: elfin_description/urdf/elfin10.urdf.xacro (robot description, xacro)
@@ -16,5 +16,5 @@
       link="elfin_base_link" />
   </joint>
-  <link name="elfin_base_link"/>
+   <link name="elfin_base_link"/>
   <joint name="elfin_base_joint" type="fixed">
     <origin
@@ -26,34 +26,41 @@
       link="elfin_base" />
   </joint>
-  <link
+   <link
     name="elfin_base">
     <inertial>
       <origin
-        xyz="0.00029790659221 0.00271788312044 0.0274159041935"
-        rpy="0 0 0"/>
-      <mass value="${0.890680700037*density}"/>
-      <inertia
-      ixx="${0.00287631*density}" ixy="${1.617e-05*density}" ixz="${3.38e-06*density}"
-      iyy="${0.00304792*density}" iyz="${2.79e-05*density}"
-      izz="${0.00537429*density}"/>
-    </inertial>
-    <visual>
-      <origin
-        xyz="0 0 0"
-        rpy="0 0 0" />
-      <geometry>
-        <mesh
-          filename="package://elfin_description/meshes/elfin10/elfin_base.STL" />
-      </geometry>
-      <material
-        name="metal_white"/>
-    </visual>
-    <collision>
-      <origin
-        xyz="0 0 0"
-        rpy="0 0 0" />
-      <geometry>
-        <mesh
-          filename="package://elfin_description/meshes/elfin10/elfin_base.STL" />
+        xyz="0.000308998351988781 0.00273575090066537 0.0272874749978871"
+        rpy="0 0 0" />
+      <mass
+        value="0.885425214033795" />
+      <inertia
+        ixx="0.00268610674383135"
+        ixy="1.61497641153452E-05"
+        ixz="3.72959384780042E-06"
+        iyy="0.00301073326471619"
+        iyz="3.90037941387144E-05"
+        izz="0.00520494004071148" />
+    </inertial>
+    <visual>
+      <origin
+        xyz="0 0 0"
+        rpy="0 0 0" />
+      <geometry>
+        <mesh
+          filename="package://elfin_description/meshes/elfin10/elfin_base_link.STL" />
+      </geometry>
+      <material
+        name="">
+        <color
+          rgba="1 1 1 1" />
+      </material>
+    </visual>
+    <collision>
+      <origin
+        xyz="0 0 0"
+        rpy="0 0 0" />
+      <geometry>
+        <mesh
+          filename="package://elfin_description/meshes/elfin10/elfin_base_link.STL" />
       </geometry>
     </collision>
@@ -63,11 +70,15 @@
     <inertial>
       <origin
-        xyz="-0.0255519176997 0.195603533565 1.68999482169e-05"
-        rpy="0 0 0"/>
-      <mass value="${5.04797690664*density}"/>
-      <inertia
-      ixx="${0.03982126*density}" ixy="${0.00844769*density}" ixz="${-4.29e-06*density}"
-      iyy="${0.02114179*density}" iyz="${-2.23e-06*density}"
-      izz="${0.04547525*density}"/>
+        xyz="-0.0256023262243377 -1.62602847268471E-05 0.0821397524271189"
+        rpy="0 0 0" />
+      <mass
+        value="5.0666551243434" />
+      <inertia
+        ixx="0.038977097970591"
+        ixy="6.08838549359665E-06"
+        ixz="0.00975553606854457"
+        iyy="0.0431999258303973"
+        iyz="2.92439974857155E-06"
+        izz="0.0198076858553278" />
     </inertial>
     <visual>
@@ -80,5 +91,8 @@
       </geometry>
       <material
-        name="metal"/>
+        name="">
+        <color
+          rgba="1 1 1 1" />
+      </material>
     </visual>
     <collision>
@@ -96,6 +110,6 @@
     type="revolute">
     <origin
-      xyz="0 0 0"
-      rpy="${PI/2} 0 0" />
+      xyz="0 0 0.1135"
+      rpy="0 0 0" />
     <parent
       link="elfin_base" />
@@ -103,5 +117,5 @@
       link="elfin_link1" />
     <axis
-      xyz="0 1 0" />
+      xyz="0 0 1" />
     <limit
       lower="-3.14"
@@ -114,11 +128,15 @@
     <inertial>
       <origin
-        xyz="-0.0589642426226 0.20968040657 -5.33587812464e-06"
-        rpy="0 0 0"/>
-      <mass value="${1.66596877354*density}"/>
-      <inertia
-      ixx="${0.052412*density}" ixy="${-0.00219612*density}" ixz="${-1.07e-06*density}"
-      iyy="${0.00434323*density}" iyz="${-1.255e-05*density}"
-      izz="${0.05107023*density}"/>
+        xyz="-0.00733875204652666 -0.203204758586133 0.0410958376319429"
+        rpy="0 0 0" />
+      <mass
+        value="1.67187821121901" />
+      <inertia
+        ixx="0.0439464748772139"
+        ixy="-9.56963727666492E-06"
+        ixz="-5.81264740217952E-07"
+        iyy="0.00419748327993436"
+        iyz="-0.00166261669205279"
+        izz="0.0454846532898179" />
     </inertial>
     <visual>
@@ -131,5 +149,8 @@
       </geometry>
       <material
-        name="metal_grey"/>
+        name="">
+        <color
+          rgba="1 1 1 1" />
+      </material>
     </visual>
     <collision>
@@ -147,6 +168,6 @@
     type="revolute">
     <origin
-      xyz="-0.084469 0.26 0"
-      rpy="0 0 0" />
+      xyz="-0.102499985410128 0.00732886700183363 0.153244350761449"
+      rpy="-1.5707963267949 0 1.5707963267949" />
     <parent
       link="elfin_link1" />
@@ -154,5 +175,5 @@
       link="elfin_link2" />
     <axis
-      xyz="-1 0 0" />
+      xyz="0 0 1" />
     <limit
       lower="-2.35"
@@ -165,11 +186,15 @@
     <inertial>
       <origin
-        xyz="0.0625690665762 -0.0521846187635 2.58799082907e-05"
-        rpy="0 0 0"/>
-      <mass value="${2.51986584925*density}"/>
-      <inertia
-      ixx="${0.01259396*density}" ixy="${0.00288795*density}" ixz="${-1.16e-06*density}"
-      iyy="${0.00707893*density}" iyz="${-2.15e-06*density}"
-      izz="${0.01493778*density}"/>
+        xyz="2.41698443355562E-05 -0.0521743520401219 -0.0560418101258959"
+        rpy="0 0 0" />
+      <mass
+        value="2.52833871519162" />
+      <inertia
+        ixx="0.0139633942538435"
+        ixy="-3.226921129389E-06"
+        ixz="2.15712479037642E-06"
+        iyy="0.00648774151674613"
+        iyz="-0.00342599914450158"
+        izz="0.0122349254525393" />
     </inertial>
     <visual>
@@ -182,5 +207,8 @@
       </geometry>
       <material
-        name="metal"/>
+        name="">
+        <color
+          rgba="1 1 1 1" />
+      </material>
     </visual>
     <collision>
@@ -198,6 +226,6 @@
     type="revolute">
     <origin
-      xyz="0 0.48 0"
-      rpy="${PI} 0 0" />
+      xyz="-0.00732886700183536 -0.473255648966734 -0.0245000000000048"
+      rpy="0 0 0" />
     <parent
       link="elfin_link2" />
@@ -205,5 +233,5 @@
       link="elfin_link3" />
     <axis
-      xyz="1 0 0" />
+      xyz="0 0 -1" />
     <limit
       lower="-2.61"
@@ -216,11 +244,15 @@
     <inertial>
       <origin
-        xyz="-0.0653325107739 0.17924183252 -8.22522528991e-06"
-        rpy="0 0 0"/>
-      <mass value="${0.773882513506*density}"/>
-      <inertia
-      ixx="${0.01260891*density}" ixy="${0.00311563*density}" ixz="${5.8e-07*density}"
-      iyy="${0.00272662*density}" iyz="${-1.47e-06*density}"
-      izz="${0.01371082*density}"/>
+        xyz="-0.0655157891899572 -1.82308655212263E-05 0.15837470257518"
+        rpy="0 0 0" />
+      <mass
+        value="0.775104782083546" />
+      <inertia
+        ixx="0.0114555561082403"
+        ixy="2.19094484211439E-07"
+        ixz="0.00266651463452"
+        iyy="0.0123478082621956"
+        iyz="-1.64179944498674E-06"
+        izz="0.00252810456539086" />
     </inertial>
     <visual>
@@ -233,5 +265,8 @@
       </geometry>
       <material
-        name="metal_grey"/>
+        name="">
+        <color
+          rgba="1 1 1 1" />
+      </material>
     </visual>
     <collision>
@@ -249,6 +284,6 @@
     type="revolute">
     <origin
-      xyz="0.084469 -0.12571 0"
-      rpy="${-PI} 0 0" />
+      xyz="0 -0.146499999728183 -0.0779999855743914"
+      rpy="1.5707963267949 1.5707963267949 0" />
     <parent
       link="elfin_link3" />
@@ -256,5 +291,5 @@
       link="elfin_link4" />
     <axis
-      xyz="0 1 0" />
+      xyz="0 0 -1" />
     <limit
       lower="-3.14"
@@ -267,11 +302,15 @@
     <inertial>
       <origin
-        xyz="-0.0174451255278 -0.0377419055039 -1.41483594707e-05"
-        rpy="0 0 0"/>
-      <mass value="${1.07514483832*density}"/>
-      <inertia
-      ixx="${0.00296619*density}" ixy="${0.00072021*density}" ixz="${7.3e-07*density}"
-      iyy="${0.00182263*density}" iyz="${-3.7e-07*density}"
-      izz="${0.00372855*density}"/>
+        xyz="-7.53559402678653E-06 -0.0377654754034753 -0.047491241533565"
+        rpy="0 0 0" />
+      <mass
+        value="1.07928561350228" />
+      <inertia
+        ixx="0.00347298936695168"
+        ixy="-2.54068509779172E-07"
+        ixz="-5.75046752801039E-07"
+        iyy="0.00165141038810566"
+        iyz="-0.000859338032022029"
+        izz="0.00288851541818101" />
     </inertial>
     <visual>
@@ -284,5 +323,8 @@
       </geometry>
       <material
-        name="metal"/>
+        name="">
+        <color
+          rgba="1 1 1 1" />
+      </material>
     </visual>
     <collision>
@@ -300,6 +342,6 @@
     type="revolute">
     <origin
-      xyz="0 0.39429 0"
-      rpy="${-PI} 0 0" />
+      xyz="-0.0649999930247983 0 0.373499977225244"
+      rpy="-1.5707963267949 0 1.5707963267949" />
     <parent
       link="elfin_link4" />
@@ -307,5 +349,5 @@
       link="elfin_link5" />
     <axis
-      xyz="1 0 0" />
+      xyz="0 0 -1" />
     <limit
       lower="-2.56"
@@ -318,11 +360,15 @@
     <inertial>
       <origin
-        xyz="0.00115745849085 0.0594966864835 0.000222299836983"
-        rpy="0 0 0"/>
-      <mass value="${0.184390264995*density}"/>
-      <inertia
-      ixx="${0.00018992*density}" ixy="${4.57e-06*density}" ixz="${-1.29e-06*density}"
-      iyy="${0.0002179*density}" iyz="${8.3e-07*density}"
-      izz="${0.00020144*density}"/>
+        xyz="-0.00817384445024986 9.28078187108763E-05 0.0394638017467175"
+        rpy="0 0 0" />
+      <mass
+        value="0.119882046423882" />
+      <inertia
+        ixx="8.12013652521768E-05"
+        ixy="2.08687521048734E-07"
+        ixz="-2.2234968672821E-06"
+        iyy="8.35696503343738E-05"
+        iyz="1.10054365931951E-09"
+        izz="0.000140099518584709" />
     </inertial>
     <visual>
@@ -335,5 +381,8 @@
       </geometry>
       <material
-        name="metal_white"/>
+        name="">
+        <color
+          rgba="1 1 1 1" />
+      </material>
     </visual>
     <collision>
@@ -351,6 +400,6 @@
     type="revolute">
     <origin
-      xyz="0 -0.111 0"
-      rpy="${PI} 0 0" />
+      xyz="0 -0.105 -0.065"
+      rpy="1.5708 1.5708 0" />
     <parent
       link="elfin_link5" />
@@ -358,5 +407,5 @@
       link="elfin_link6" />
     <axis
-      xyz="0 1 0" />
+      xyz="0 0 1" />
     <limit
       lower="-3.14"
@@ -365,9 +414,11 @@
       velocity="1.57" />
   </joint>
-  <link name="elfin_end_link"/>
-  <joint name="elfin_end_joint" type="fixed">
-    <origin
-      xyz="0 0.089 0"
-      rpy="${-PI/2} ${-PI/2} 0" />
+   <link name="elfin_end_link"/>
+  <joint
+    name="elfin_end_joint"
+    type="fixed">
+    <origin
+      xyz="-0.000370495118397286 0.000153464102833181 0.0629999999999997"
+      rpy="0 0 -0.0122082043644551" />
     <parent
       link="elfin_link6" />

File: elfin_description/urdf/elfin3.urdf.xacro (robot description, xacro)
@@ -30,6 +30,6 @@
     <inertial>
       <origin
-        xyz="0.000476057496448 -0.00609847721085 0.0271227961552"
-        rpy="0 0 0"/>
+        xyz="8.7997E-06 0.00045737 0.025376"
+        rpy="0 0 0" />
       <mass value="${0.432503561632*density}"/>
       <inertia
@@ -63,6 +63,6 @@
     <inertial>
       <origin
-        xyz="-0.0192425632808 0.120157543892 -2.05350524914e-05"
-        rpy="0 0 0"/>
+        xyz="-0.02107 1.8203E-05 0.070829"
+        rpy="0 0 0" />
       <mass value="${1.52001312557*density}"/>
       <inertia
@@ -96,6 +96,6 @@
     type="revolute">
     <origin
-      xyz="0 0 0.031"
-      rpy="${PI/2} 0 0" />
+      xyz="0 0 0.0745"
+      rpy="0 0 0" />
     <parent
       link="elfin_base" />
@@ -103,5 +103,5 @@
       link="elfin_link1" />
     <axis
-      xyz="0 1 0" />
+      xyz="0 0 1" />
     <limit
       lower="-3.14"
@@ -114,6 +114,6 @@
     <inertial>
       <origin
-        xyz="-0.0363359816546 0.121774838175 -3.84046105722e-05"
-        rpy="0 0 0"/>
+        xyz="-2.0075E-05 0.12327 0.036666"
+        rpy="0 0 0" />
       <mass value="${0.519672255247*density}"/>
       <inertia
@@ -147,6 +147,6 @@
     type="revolute">
     <origin
-      xyz="-0.068808 0.1615 0"
-      rpy="0 0 0" />
+      xyz="-0.072 0 0.117"
+      rpy="1.5708 0 -1.5708" />
     <parent
       link="elfin_link1" />
@@ -154,5 +154,5 @@
       link="elfin_link2" />
     <axis
-      xyz="-1 0 0" />
+      xyz="0 0 1" />
     <limit
       lower="-2.35"
@@ -165,6 +165,6 @@
     <inertial>
       <origin
-        xyz="0.0513625008301 -0.0377418700977 -1.41484011876e-05"
-        rpy="0 0 0"/>
+        xyz="9.6224E-06 0.042461 -0.044165"
+        rpy="0 0 0" />
       <mass value="${1.07514585114*density}"/>
       <inertia
@@ -198,6 +198,6 @@
     type="revolute">
     <origin
-      xyz="0 0.266 0"
-      rpy="${-PI} 0 0" />
+      xyz="0 0.266 -0.007"
+      rpy="0 0 0" />
     <parent
       link="elfin_link2" />
@@ -205,5 +205,5 @@
       link="elfin_link3" />
     <axis
-      xyz="1 0 0" />
+      xyz="0 0 -1" />
     <limit
       lower="-2.61"
@@ -216,6 +216,6 @@
     <inertial>
       <origin
-        xyz="-0.0580853772834 0.10002233137 -3.45203877103e-06"
-        rpy="0 0 0"/>
+        xyz="-0.055318 3.0677E-06 0.099673"
+        rpy="0 0 0" />
       <mass value="${0.37026646381*density}"/>
       <inertia
@@ -249,6 +249,6 @@
     type="revolute">
     <origin
-      xyz="0.068808 -0.10523 0"
-      rpy="${PI} 0 0" />
+      xyz="0 0.105 -0.065"
+      rpy="0 1.57 1.570" />
     <parent
       link="elfin_link3" />
@@ -256,5 +256,5 @@
       link="elfin_link4" />
     <axis
-      xyz="0 1 0" />
+      xyz="0 0 -1" />
     <limit
       lower="-3.14"
@@ -267,6 +267,6 @@
     <inertial>
       <origin
-        xyz="-0.0158710385319 -0.0365214098995 4.94388107361e-07"
-        rpy="0 0 0"/>
+        xyz="3.7144E-06 0.039279 -0.043638"
+        rpy="0 0 0" />
       <mass value="${0.807027243448*density}"/>
       <inertia
@@ -300,6 +300,6 @@
     type="revolute">
     <origin
-      xyz="0 0.21877 0"
-      rpy="${-PI} 0 0" />
+      xyz="-0.06025 0 0.219"
+      rpy="1.5708 0 -1.5708" />
     <parent
       link="elfin_link4" />
@@ -307,5 +307,5 @@
       link="elfin_link5" />
     <axis
-      xyz="1 0 0" />
+      xyz="0 0 -1" />
     <limit
       lower="-2.56"
@@ -318,5 +318,5 @@
     <inertial>
       <origin
-        xyz="-0.0009237 -0.042691 -0.0003367"
+        xyz="-0.0070896 -0.00016176 0.034853"
         rpy="0 0 0" />
       <mass value="${0.147312*density}"/>
@@ -351,6 +351,6 @@
     type="revolute">
     <origin
-      xyz="0 -0.1065 0"
-      rpy="${-PI} 0 ${-PI}" />
+      xyz="0 0.10075 -0.06025"
+      rpy="0 1.5645 1.5734" />
     <parent
       link="elfin_link5" />
@@ -358,5 +358,5 @@
       link="elfin_link6" />
     <axis
-      xyz="0 -1 0" />
+      xyz="0 0 -1" />
     <limit
       lower="-3.14"
@@ -368,6 +368,6 @@
   <joint name="elfin_end_joint" type="fixed">
     <origin
-      xyz="0 -0.091 0"
-      rpy="${PI/2} ${-PI/2} 0" />
+      xyz="0 0 0.059251"
+      rpy="0.0025901 0.006253 0" />
     <parent
       link="elfin_link6" />

File: elfin_description/urdf/elfin5.urdf.xacro (robot description, xacro)
@@ -30,5 +30,5 @@
     <inertial>
       <origin
-        xyz="0.000209 0.001319 0.025619"
+         xyz="0.00022102 0.0013404 0.025529"
         rpy="0 0 0" />
       <mass value="${0.690521*density}"/>
@@ -63,5 +63,5 @@
     <inertial>
       <origin
-        xyz="-0.0217491 0.1389011 0.0000125"
+        xyz="-0.021815 -1.1609E-05 0.095394"
         rpy="0 0 0" />
       <mass value="${2.576772*density}"/>
@@ -96,6 +96,6 @@
     type="revolute">
     <origin
-      xyz="0 0 0.03"
-      rpy="${PI/2} 0 0" />
+      xyz="0 0 0.0735"
+      rpy="0 0 0" />
     <parent
       link="elfin_base" />
@@ -103,5 +103,5 @@
       link="elfin_link1" />
     <axis
-      xyz="0 1 0" />
+      xyz="0 0 1" />
     <limit
       lower="-3.14"
@@ -114,5 +114,5 @@
     <inertial>
       <origin
-        xyz="-0.0522485 0.1580101 -0.0000003"
+        xyz="-0.15508 0.031021 0.052499"
         rpy="0 0 0" />
       <mass value="${1.208607*density}"/>
@@ -147,12 +147,12 @@
     type="revolute">
     <origin
-      xyz="-0.078069 0.19 0"
-      rpy="0 0 0" />
+      xyz="-0.078 0 0.1465"
+      rpy="1.5708 1.3734 -1.5708" />
     <parent
       link="elfin_link1" />
     <child
       link="elfin_link2" />
-    <axis
-      xyz="-1 0 0" />
+   <axis
+      xyz="0 0 1" />
     <limit
       lower="-2.35"
@@ -165,5 +165,5 @@
     <inertial>
       <origin
-        xyz="0.0587091 -0.0414608 -0.0000210"
+        xyz="1.1184E-05 0.041481 -0.052586"
         rpy="0 0 0" />
       <mass value="${1.525883*density}"/>
@@ -198,6 +198,6 @@
     type="revolute">
     <origin
-      xyz="0 0.38 0"
-      rpy="${PI} 0 0" />
+      xyz="-0.37262 0.074541 -0.0060028"
+      rpy="0 0 1.3734" />
     <parent
       link="elfin_link2" />
@@ -205,9 +205,9 @@
       link="elfin_link3" />
     <axis
-      xyz="1 0 0" />
+      xyz="0 0 -1" />
     <limit
       lower="-2.61"
       upper="2.61"
-      effort="104"
+      effort="200"
       velocity="1.57" />
   </joint>
@@ -216,5 +216,5 @@
     <inertial>
       <origin
-        xyz="-0.0587964 0.1436154 -0.0000478"
+        xyz="-0.058961 3.7945E-05 0.13807"
         rpy="0 0 0" />
       <mass value="${0.475026*density}"/>
@@ -249,6 +249,6 @@
     type="revolute">
     <origin
-      xyz="0.078069 -0.11342 0"
-      rpy="${-PI} 0 0" />
+      xyz="0 0.119 -0.072"
+      rpy="0 1.5708 1.5708" />
     <parent
       link="elfin_link3" />
@@ -256,5 +256,5 @@
       link="elfin_link4" />
     <axis
-      xyz="0 1 0" />
+      xyz="0 0 -1" />
     <limit
       lower="-3.14"
@@ -267,5 +267,5 @@
     <inertial>
       <origin
-        xyz="-0.0159154 -0.0365660 0.0000004"
+        xyz="3.4043E-06 -0.036593 -0.044531"
         rpy="0 0 0" />
       <mass value="${0.808399*density}"/>
@@ -300,12 +300,12 @@
     type="revolute">
     <origin
-      xyz="0 0.30658 0"
-      rpy="${-PI} 0 0" />
+      xyz="-0.0605 0 0.301"
+      rpy="-1.5708 0 1.5708" />
     <parent
       link="elfin_link4" />
     <child
       link="elfin_link5" />
-    <axis
-      xyz="1 0 0" />
+   <axis
+      xyz="0 0 -1" />
     <limit
       lower="-2.56"
@@ -318,5 +318,5 @@
     <inertial>
       <origin
-        xyz="-0.0009237 -0.042691 -0.0003367"
+        xyz="-0.007255 -3.2028E-05 0.033062"
         rpy="0 0 0" />
       <mass value="${0.147312*density}"/>
@@ -351,6 +351,6 @@
     type="revolute">
     <origin
-      xyz="0 -0.1065 0"
-      rpy="0 0 0" />
+      xyz="0 -0.1005 -0.0605"
+      rpy="1.5708 1.5708 0" />
     <parent
       link="elfin_link5" />
@@ -358,5 +358,5 @@
       link="elfin_link6" />
     <axis
-      xyz="0 -1 0" />
+      xyz="0 0 1" />
     <limit
       lower="-3.14"
@@ -368,6 +368,6 @@
   <joint name="elfin_end_joint" type="fixed">
     <origin
-      xyz="0 -0.0735 0"
-      rpy="${PI/2} ${PI/2} 0" />
+      xyz="0 0 0.0485"
+      rpy="0 0 0" />
     <parent
       link="elfin_link6" />
