Commit message: update

File: elfin_description/urdf/elfin10.urdf.xacro (robot description, xacro)
@@ -10,5 +10,5 @@
     <origin
       xyz="0 0 0"
-      rpy="0 0 0" />
+      rpy="0 0 -1.5708" />
     <parent
       link="world" />
@@ -26,19 +26,19 @@
       link="elfin_base" />
   </joint>
-   <link
+  <link
     name="elfin_base">
     <inertial>
       <origin
-        xyz="0.000308998351988781 0.00273575090066537 0.0272874749978871"
-        rpy="0 0 0" />
-      <mass
-        value="0.885425214033795" />
-      <inertia
-        ixx="0.00268610674383135"
-        ixy="1.61497641153452E-05"
-        ixz="3.72959384780042E-06"
-        iyy="0.00301073326471619"
-        iyz="3.90037941387144E-05"
-        izz="0.00520494004071148" />
+        xyz="-0.00272891148525253 0.000307855470977014 0.0272857003429058"
+        rpy="0 0 0" />
+      <mass
+        value="0.885322892252566" />
+      <inertia
+        ixx="0.00301072999783137"
+        ixy="-1.61177742996604E-05"
+        ixz="-3.9001744857601E-05"
+        iyy="0.0026859684784965"
+        iyz="3.74127558541537E-06"
+        izz="0.00520484836475965" />
     </inertial>
     <visual>
@@ -53,4 +53,44 @@
         name="">
         <color
+          rgba="0.792156862745098 0.819607843137255 0.929411764705882 1" />
+      </material>
+    </visual>
+    <collision>
+      <origin
+        xyz="0 0 0"
+        rpy="0 0 0" />
+      <geometry>
+        <mesh
+          filename="package://elfin_description/meshes/elfin10/elfin_base_link.STL" />
+      </geometry>
+    </collision>
+  </link>
+  <link
+    name="elfin_link1">
+    <inertial>
+      <origin
+        xyz="1.64450419081555E-05 -0.0256037445106889 0.116231470679274"
+        rpy="0 0 0" />
+      <mass
+        value="5.06676664437865" />
+      <inertia
+        ixx="0.0432021422624639"
+        ixy="-5.87315615826586E-06"
+        ixz="-3.3817285662756E-06"
+        iyy="0.0389769463442445"
+        iyz="0.00975755293023606"
+        izz="0.0198084067505502" />
+    </inertial>
+    <visual>
+      <origin
+        xyz="0 0 0"
+        rpy="0 0 0" />
+      <geometry>
+        <mesh
+          filename="package://elfin_description/meshes/elfin10/elfin_link1.STL" />
+      </geometry>
+      <material
+        name="">
+        <color
           rgba="1 1 1 1" />
       </material>
@@ -62,46 +102,6 @@
       <geometry>
         <mesh
-          filename="package://elfin_description/meshes/elfin10/elfin_base_link.STL" />
-      </geometry>
-    </collision>
-  </link>
-  <link
-    name="elfin_link1">
-    <inertial>
-      <origin
-        xyz="-0.0256023262243377 -1.62602847268471E-05 0.0821397524271189"
-        rpy="0 0 0" />
-      <mass
-        value="5.0666551243434" />
-      <inertia
-        ixx="0.038977097970591"
-        ixy="6.08838549359665E-06"
-        ixz="0.00975553606854457"
-        iyy="0.0431999258303973"
-        iyz="2.92439974857155E-06"
-        izz="0.0198076858553278" />
-    </inertial>
-    <visual>
-      <origin
-        xyz="0 0 0"
-        rpy="0 0 0" />
-      <geometry>
-        <mesh
           filename="package://elfin_description/meshes/elfin10/elfin_link1.STL" />
       </geometry>
-      <material
-        name="">
-        <color
-          rgba="1 1 1 1" />
-      </material>
-    </visual>
-    <collision>
-      <origin
-        xyz="0 0 0"
-        rpy="0 0 0" />
-      <geometry>
-        <mesh
-          filename="package://elfin_description/meshes/elfin10/elfin_link1.STL" />
-      </geometry>
     </collision>
   </link>
@@ -110,5 +110,5 @@
     type="revolute">
     <origin
-      xyz="0 0 0.1135"
+      xyz="0 0 0.0794"
       rpy="0 0 0" />
     <parent
@@ -121,5 +121,5 @@
       lower="-3.14"
       upper="3.14"
-      effort="420"
+      effort="104"
       velocity="1.57" />
   </joint>
@@ -128,15 +128,15 @@
     <inertial>
       <origin
-        xyz="-0.00733875204652666 -0.203204758586133 0.0410958376319429"
-        rpy="0 0 0" />
-      <mass
-        value="1.67187821121901" />
-      <inertia
-        ixx="0.0439464748772139"
-        ixy="-9.56963727666492E-06"
-        ixz="-5.81264740217952E-07"
-        iyy="0.00419748327993436"
-        iyz="-0.00166261669205279"
-        izz="0.0454846532898179" />
+        xyz="6.76058799303212E-06 -0.042999875819422 0.209938025941438"
+        rpy="0 0 0" />
+      <mass
+        value="1.67177851395468" />
+      <inertia
+        ixx="0.0439485446845192"
+        ixy="-4.52807636811865E-07"
+        ixz="-7.43339382852812E-06"
+        iyy="0.0454864353408678"
+        iyz="-0.0016627192868139"
+        izz="0.00419718886154138" />
     </inertial>
     <visual>
@@ -151,5 +151,5 @@
         name="">
         <color
-          rgba="1 1 1 1" />
+          rgba="0.501960784313725 0.501960784313725 0.501960784313725 1" />
       </material>
     </visual>
@@ -168,6 +168,6 @@
     type="revolute">
     <origin
-      xyz="-0.102499985410128 0.00732886700183363 0.153244350761449"
-      rpy="-1.5707963267949 0 1.5707963267949" />
+      xyz="0 -0.1006 0.1806"
+      rpy="0 0 0" />
     <parent
       link="elfin_link1" />
@@ -175,9 +175,9 @@
       link="elfin_link2" />
     <axis
-      xyz="0 0 1" />
+      xyz="0 -1 0" />
     <limit
       lower="-2.35"
       upper="2.35"
-      effort="420"
+      effort="104"
       velocity="1.57" />
   </joint>
@@ -186,15 +186,15 @@
     <inertial>
       <origin
-        xyz="2.41698443355562E-05 -0.0521743520401219 -0.0560418101258959"
-        rpy="0 0 0" />
-      <mass
-        value="2.52833871519162" />
-      <inertia
-        ixx="0.0139633942538435"
-        ixy="-3.226921129389E-06"
-        ixz="2.15712479037642E-06"
-        iyy="0.00648774151674613"
-        iyz="-0.00342599914450158"
-        izz="0.0122349254525393" />
+        xyz="-2.62996059291557E-05 0.0490394097580479 0.052175062906049"
+        rpy="0 0 0" />
+      <mass
+        value="2.52843012692852" />
+      <inertia
+        ixx="0.0139637252708319"
+        ixy="2.19112531145417E-06"
+        ixz="-3.30099393077099E-06"
+        iyy="0.0122350897234042"
+        iyz="-0.00342609019238153"
+        izz="0.00648764255835148" />
     </inertial>
     <visual>
@@ -226,5 +226,5 @@
     type="revolute">
     <origin
-      xyz="-0.00732886700183536 -0.473255648966734 -0.0245000000000048"
+      xyz="0 0.0296 0.48"
       rpy="0 0 0" />
     <parent
@@ -233,9 +233,9 @@
       link="elfin_link3" />
     <axis
-      xyz="0 0 -1" />
+      xyz="0 1 0" />
     <limit
       lower="-2.61"
       upper="2.61"
-      effort="200"
+      effort="69"
       velocity="1.57" />
   </joint>
@@ -244,15 +244,15 @@
     <inertial>
       <origin
-        xyz="-0.0655157891899572 -1.82308655212263E-05 0.15837470257518"
-        rpy="0 0 0" />
-      <mass
-        value="0.775104782083546" />
-      <inertia
-        ixx="0.0114555561082403"
-        ixy="2.19094484211439E-07"
-        ixz="0.00266651463452"
-        iyy="0.0123478082621956"
-        iyz="-1.64179944498674E-06"
-        izz="0.00252810456539086" />
+        xyz="7.16230692529086E-06 -0.0655290443401757 0.159896102785824"
+        rpy="0 0 0" />
+      <mass
+        value="0.77472632829127" />
+      <inertia
+        ixx="0.0123453730002939"
+        ixy="5.3931985013663E-08"
+        ixz="6.96327319489119E-07"
+        iyy="0.0114525775167076"
+        iyz="0.00266638141144531"
+        izz="0.00252781952691956" />
     </inertial>
     <visual>
@@ -267,5 +267,5 @@
         name="">
         <color
-          rgba="1 1 1 1" />
+          rgba="0.501960784313725 0.501960784313725 0.501960784313725 1" />
       </material>
     </visual>
@@ -284,126 +284,10 @@
     type="revolute">
     <origin
-      xyz="0 -0.146499999728183 -0.0779999855743914"
-      rpy="1.5707963267949 1.5707963267949 0" />
+      xyz="0 0.071 0.145"
+      rpy="0 0 0" />
     <parent
       link="elfin_link3" />
     <child
       link="elfin_link4" />
-    <axis
-      xyz="0 0 -1" />
-    <limit
-      lower="-3.14"
-      upper="3.14"
-      effort="200"
-      velocity="1.57" />
-  </joint>
-  <link
-    name="elfin_link5">
-    <inertial>
-      <origin
-        xyz="-7.53559402678653E-06 -0.0377654754034753 -0.047491241533565"
-        rpy="0 0 0" />
-      <mass
-        value="1.07928561350228" />
-      <inertia
-        ixx="0.00347298936695168"
-        ixy="-2.54068509779172E-07"
-        ixz="-5.75046752801039E-07"
-        iyy="0.00165141038810566"
-        iyz="-0.000859338032022029"
-        izz="0.00288851541818101" />
-    </inertial>
-    <visual>
-      <origin
-        xyz="0 0 0"
-        rpy="0 0 0" />
-      <geometry>
-        <mesh
-          filename="package://elfin_description/meshes/elfin10/elfin_link5.STL" />
-      </geometry>
-      <material
-        name="">
-        <color
-          rgba="1 1 1 1" />
-      </material>
-    </visual>
-    <collision>
-      <origin
-        xyz="0 0 0"
-        rpy="0 0 0" />
-      <geometry>
-        <mesh
-          filename="package://elfin_description/meshes/elfin10/elfin_link5.STL" />
-      </geometry>
-    </collision>
-  </link>
-  <joint
-    name="elfin_joint5"
-    type="revolute">
-    <origin
-      xyz="-0.0649999930247983 0 0.373499977225244"
-      rpy="-1.5707963267949 0 1.5707963267949" />
-    <parent
-      link="elfin_link4" />
-    <child
-      link="elfin_link5" />
-    <axis
-      xyz="0 0 -1" />
-    <limit
-      lower="-2.56"
-      upper="2.56"
-      effort="69"
-      velocity="1.57" />
-  </joint>
-  <link
-    name="elfin_link6">
-    <inertial>
-      <origin
-        xyz="-0.00817384445024986 9.28078187108763E-05 0.0394638017467175"
-        rpy="0 0 0" />
-      <mass
-        value="0.119882046423882" />
-      <inertia
-        ixx="8.12013652521768E-05"
-        ixy="2.08687521048734E-07"
-        ixz="-2.2234968672821E-06"
-        iyy="8.35696503343738E-05"
-        iyz="1.10054365931951E-09"
-        izz="0.000140099518584709" />
-    </inertial>
-    <visual>
-      <origin
-        xyz="0 0 0"
-        rpy="0 0 0" />
-      <geometry>
-        <mesh
-          filename="package://elfin_description/meshes/elfin10/elfin_link6.STL" />
-      </geometry>
-      <material
-        name="">
-        <color
-          rgba="1 1 1 1" />
-      </material>
-    </visual>
-    <collision>
-      <origin
-        xyz="0 0 0"
-        rpy="0 0 0" />
-      <geometry>
-        <mesh
-          filename="package://elfin_description/meshes/elfin10/elfin_link6.STL" />
-      </geometry>
-    </collision>
-  </link>
-  <joint
-    name="elfin_joint6"
-    type="revolute">
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
File: elfin_description/urdf/elfin3.urdf.xacro (robot description, xacro)
@@ -10,5 +10,5 @@
     <origin
       xyz="0 0 0"
-      rpy="0 0 0" />
+      rpy="0 0 -1.5708" />
     <parent
       link="world" />
@@ -26,34 +26,41 @@
       link="elfin_base" />
   </joint>
-  <link
+ <link
     name="elfin_base">
     <inertial>
       <origin
-        xyz="8.7997E-06 0.00045737 0.025376"
-        rpy="0 0 0" />
-      <mass value="${0.432503561632*density}"/>
-      <inertia
-      ixx="${0.00107966*density}" ixy="${6.43e-06*density}" ixz="${1.97e-06*density}"
-      iyy="${0.00089216*density}" iyz="${-1.269e-05*density}"
-      izz="${0.00174712*density}"/>
-    </inertial>
-    <visual>
-      <origin
-        xyz="0 0 0"
-        rpy="0 0 0" />
-      <geometry>
-        <mesh
-          filename="package://elfin_description/meshes/elfin3/elfin_base.STL" />
-      </geometry>
-      <material
-        name="metal_white"/>
-    </visual>
-    <collision>
-      <origin
-        xyz="0 0 0"
-        rpy="0 0 0" />
-      <geometry>
-        <mesh
-          filename="package://elfin_description/meshes/elfin3/elfin_base.STL" />
+        xyz="0.00425937844813294 -0.000389571231902992 0.00274262778667868"
+        rpy="0 0 0" />
+      <mass
+        value="0.0268461773395224" />
+      <inertia
+        ixx="2.66341322206443E-05"
+        ixy="5.51640996553045E-08"
+        ixz="2.21112209410463E-12"
+        iyy="2.67121402645769E-05"
+        iyz="-3.17722287525956E-12"
+        izz="5.30011200382481E-05" />
+    </inertial>
+    <visual>
+      <origin
+        xyz="0 0 0"
+        rpy="0 0 0" />
+      <geometry>
+        <mesh
+          filename="package://elfin_description/meshes/elfin3/base_link.STL" />
+      </geometry>
+      <material
+        name="">
+        <color
+          rgba="0.686274509803922 0.686274509803922 0.686274509803922 1" />
+      </material>
+    </visual>
+    <collision>
+      <origin
+        xyz="0 0 0"
+        rpy="0 0 0" />
+      <geometry>
+        <mesh
+          filename="package://elfin_description/meshes/elfin3/base_link.STL" />
       </geometry>
     </collision>
@@ -63,11 +70,15 @@
     <inertial>
       <origin
-        xyz="-0.02107 1.8203E-05 0.070829"
-        rpy="0 0 0" />
-      <mass value="${1.52001312557*density}"/>
-      <inertia
-      ixx="${0.00523815*density}" ixy="${0.00122593*density}" ixz="${-1.6e-07*density}"
-      iyy="${0.00315471*density}" iyz="${-6.4e-07*density}"
-      izz="${0.00646649*density}"/>
+        xyz="-1.11474311817293E-05 -0.019295238440266 0.081643413279284"
+        rpy="0 0 0" />
+      <mass
+        value="1.52628719338585" />
+      <inertia
+        ixx="0.006028902112623"
+        ixy="-5.48816506919481E-07"
+        ixz="-2.73302311360408E-07"
+        iyy="0.00509895338088794"
+        iyz="0.00146640275062038"
+        izz="0.0028687934642813" />
     </inertial>
     <visual>
@@ -80,5 +91,8 @@
       </geometry>
       <material
-        name="metal"/>
+        name="">
+        <color
+          rgba="0.772549019607843 0.752941176470588 0.733333333333333 1" />
+      </material>
     </visual>
     <collision>
@@ -96,5 +110,5 @@
     type="revolute">
     <origin
-      xyz="0 0 0.0745"
+      xyz="0 0 0.0695"
       rpy="0 0 0" />
     <parent
@@ -114,11 +128,15 @@
     <inertial>
       <origin
-        xyz="-2.0075E-05 0.12327 0.036666"
-        rpy="0 0 0" />
-      <mass value="${0.519672255247*density}"/>
-      <inertia
-      ixx="${0.00564813*density}" ixy="${-0.00026473*density}" ixz="${0.0*density}"
-      iyy="${0.00053594*density}" iyz="${1.29e-06*density}"
-      izz="${0.00545618*density}"/>
+        xyz="-3.09813419838078E-05 -0.0392725728395098 0.121906520746464"
+        rpy="0 0 0" />
+      <mass
+        value="0.519379765009091" />
+      <inertia
+        ixx="0.00462941997584524"
+        ixy="9.53033193206284E-08"
+        ixz="1.89958745191593E-06"
+        iyy="0.00485416387879526"
+        iyz="-0.00019166604937554"
+        izz="0.000506978474454832" />
     </inertial>
     <visual>
@@ -131,5 +149,8 @@
       </geometry>
       <material
-        name="metal_grey"/>
+        name="">
+        <color
+          rgba="0.501960784313725 0.501960784313725 0.501960784313725 1" />
+      </material>
     </visual>
     <collision>
@@ -147,6 +168,6 @@
     type="revolute">
     <origin
-      xyz="-0.072 0 0.117"
-      rpy="1.5708 0 -1.5708" />
+      xyz="0 -0.066 0.123"
+      rpy="0 0 0" />
     <parent
       link="elfin_link1" />
@@ -154,10 +175,10 @@
       link="elfin_link2" />
     <axis
-      xyz="0 0 1" />
+      xyz="0 -1 0" />
     <limit
       lower="-2.35"
       upper="2.35"
       effort="104"
-      velocity="1.57" />
+      velocity="1.27" />
   </joint>
   <link
@@ -165,11 +186,15 @@
     <inertial>
       <origin
-        xyz="9.6224E-06 0.042461 -0.044165"
-        rpy="0 0 0" />
-      <mass value="${1.07514585114*density}"/>
-      <inertia
-      ixx="${0.00296619*density}" ixy="${0.00072021*density}" ixz="${7.3e-07*density}"
-      iyy="${0.00182263*density}" iyz="${-3.7e-07*density}"
-      izz="${0.00372855*density}"/>
+        xyz="7.94789705792241E-06 0.0434911461385148 0.0377663456053925"
+        rpy="0 0 0" />
+      <mass
+        value="1.07924103107593" />
+      <inertia
+        ixx="0.00347290093864989"
+        ixy="-5.5219540256932E-07"
+        ixz="-1.81596933237452E-07"
+        iyy="0.0028883932232078"
+        iyz="-0.000859331225721596"
+        izz="0.00165138765596417" />
     </inertial>
     <visual>
@@ -182,5 +207,8 @@
       </geometry>
       <material
-        name="metal"/>
+        name="">
+        <color
+          rgba="1 1 1 1" />
+      </material>
     </visual>
     <collision>
@@ -198,5 +226,5 @@
     type="revolute">
     <origin
-      xyz="0 0.266 -0.007"
+      xyz="0 0.005 0.266"
       rpy="0 0 0" />
     <parent
@@ -205,5 +233,5 @@
       link="elfin_link3" />
     <axis
-      xyz="0 0 -1" />
+      xyz="0 1 0" />
     <limit
       lower="-2.61"
@@ -216,11 +244,15 @@
     <inertial>
       <origin
-        xyz="-0.055318 3.0677E-06 0.099673"
-        rpy="0 0 0" />
-      <mass value="${0.37026646381*density}"/>
-      <inertia
-      ixx="${0.00238279*density}" ixy="${0.00082955*density}" ixz="${1.1e-07*density}"
-      iyy="${0.00095758*density}" iyz="${-3.2e-07*density}"
-      izz="${0.00285161*density}"/>
+        xyz="3.93948157579129E-06 -0.0583766984632963 0.104324949772583"
+        rpy="0 0 0" />
+      <mass
+        value="0.369742076927137" />
+      <inertia
+        ixx="0.00246788834863717"
+        ixy="4.99944210740992E-08"
+        ixz="-3.25489511678092E-08"
+        iyy="0.00211847372798997"
+        iyz="0.000668250395065579"
+        izz="0.000839231486986835" />
     </inertial>
     <visual>
@@ -233,5 +265,8 @@
       </geometry>
       <material
-        name="metal_grey"/>
+        name="">
+        <color
+          rgba="0.501960784313725 0.501960784313725 0.501960784313725 1" />
+      </material>
     </visual>
     <collision>
@@ -249,6 +284,6 @@
     type="revolute">
     <origin
-      xyz="0 0.105 -0.065"
-      rpy="0 1.57 1.570" />
+      xyz="0 0.061 0.101"
+      rpy="0 0 0" />
     <parent
       link="elfin_link3" />
@@ -256,5 +291,5 @@
       link="elfin_link4" />
     <axis
-      xyz="0 0 -1" />
+      xyz="0 0 1" />
     <limit
       lower="-3.14"
@@ -267,11 +302,15 @@
     <inertial>
       <origin
-        xyz="3.7144E-06 0.039279 -0.043638"
-        rpy="0 0 0" />
-      <mass value="${0.807027243448*density}"/>
-      <inertia
-      ixx="${0.00193719*density}" ixy="${0.00047145*density}" ixz="${2e-08*density}"
-      iyy="${0.00112857*density}" iyz="${-1.1e-07*density}"
-      izz="${0.00245655*density}"/>
+        xyz="-1.43602737885348E-06 0.0400732712700223 0.0365459315107893"
+        rpy="0 0 0" />
+      <mass
+        value="0.810519795979025" />
+      <inertia
+        ixx="0.00228900919014725"
+        ixy="3.53045982931884E-08"
+        ixz="2.29268789681775E-08"
+        iyy="0.00188329109495946"
+        iyz="-0.000564395858742294"
+        izz="0.00101935359998985" />
     </inertial>
     <visual>
@@ -284,5 +323,8 @@
       </geometry>
       <material
-        name="metal"/>
+        name="">
+        <color
+          rgba="0.772549019607843 0.752941176470588 0.733333333333333 1" />
+      </material>
     </visual>
     <collision>
@@ -300,6 +342,6 @@
     type="revolute">
     <origin
-      xyz="-0.06025 0 0.219"
-      rpy="1.5708 0 -1.5708" />
+      xyz="0 -0.056 0.223"
+      rpy="0 0 0" />
     <parent
       link="elfin_link4" />
@@ -307,5 +349,5 @@
       link="elfin_link5" />
     <axis
-      xyz="0 0 -1" />
+      xyz="0 1 0" />
     <limit
       lower="-2.56"
@@ -318,11 +360,15 @@
     <inertial>
       <origin
-        xyz="-0.0070896 -0.00016176 0.034853"
-        rpy="0 0 0" />
-      <mass value="${0.147312*density}"/>
-      <inertia
-      ixx="${0.00019407*density}" ixy="${1.4e-06*density}" ixz="${-2.89e-06*density}"
-      iyy="${0.00019592*density}" iyz="${5e-08*density}"
-      izz="${0.00019496*density}"/>
+        xyz="3.20814749367106E-05 -0.00725494085500073 0.0375620352744778"
+        rpy="0 0 0" />
+      <mass
+        value="0.11342880515576" />
+      <inertia
+        ixx="7.66530991301819E-05"
+        ixy="-1.83940471442645E-07"
+        ixz="-4.80914267075654E-08"
+        iyy="7.49230832326719E-05"
+        iyz="-2.34292724113658E-06"
+        izz="0.000127800839988254" />
     </inertial>
     <visual>
@@ -335,5 +381,8 @@
       </geometry>
       <material
-        name="metal_white"/>
+        name="">
+        <color
+          rgba="0.776470588235294 0.756862745098039 0.737254901960784 1" />
+      </material>
     </visual>
     <collision>
@@ -351,6 +400,6 @@
     type="revolute">
     <origin
-      xyz="0 0.10075 -0.06025"
-      rpy="0 1.5645 1.5734" />
+      xyz="0 0.056 0.096"
+      rpy="0 0 0" />
     <parent
       link="elfin_link5" />
@@ -368,6 +417,6 @@
   <joint name="elfin_end_joint" type="fixed">
     <origin
-      xyz="0 0 0.059251"
-      rpy="0.0025901 0.006253 0" />
+      xyz="0 0 0.059"
+      rpy="0 0 0" />
     <parent
       link="elfin_link6" />

File: elfin_description/urdf/elfin5.urdf.xacro (robot description, xacro)
@@ -256,5 +256,5 @@
       link="elfin_link4" />
     <axis
-      xyz="0 0 -1" />
+      xyz="0 0 1" />
     <limit
       lower="-3.14"
@@ -368,6 +368,6 @@
   <joint name="elfin_end_joint" type="fixed">
     <origin
-      xyz="0 0 0.0485"
-      rpy="0 0 0" />
+      xyz="0 0 0.0545"
+      rpy="0 0 -1.5708" />
     <parent
       link="elfin_link6" />
