Commit message: Add the elfin10_l urdf model and moveit config (remind: ikfast for elfin15 still not work)

File: elfin_description/urdf/elfin10_l.urdf.xacro (robot description, xacro)
@@ -1,4 +1,4 @@
 <robot
-  name="elfin15" xmlns:xacro="http://www.ros.org/wiki/xacro">
+  name="elfin10_l" xmlns:xacro="http://www.ros.org/wiki/xacro">
   <xacro:include filename="$(find elfin_description)/urdf/materials.xacro" />
   <xacro:include filename="$(find elfin_description)/urdf/elfin_robot.gazebo" />
@@ -28,37 +28,37 @@
     <inertial>
       <origin
-        xyz="2.654E-09 0.0003357 0.036153"
-        rpy="0 0 0" />
-      <mass
-        value="2.8356" />
-      <inertia
-        ixx="0.0097381"
-        ixy="-1.8821E-10"
-        ixz="-9.0965E-11"
-        iyy="0.0098176"
-        iyz="2.182E-05"
-        izz="0.016617" />
-    </inertial>
-    <visual>
-      <origin
-        xyz="0 0 0"
-        rpy="0 0 0" />
-      <geometry>
-        <mesh
-          filename="package://elfin_description/meshes/elfin15/elfin_base.STL" />
-      </geometry>
-      <material
-        name="">
-        <color
-          rgba="0.86667 0.86667 0.8902 1" />
-      </material>
-    </visual>
-    <collision>
-      <origin
-        xyz="0 0 0"
-        rpy="0 0 0" />
-      <geometry>
-        <mesh
-          filename="package://elfin_description/meshes/elfin15/elfin_base.STL" />
+        xyz="3.0613E-07 0.0023359 0.025589"
+        rpy="0 0 0" />
+      <mass
+        value="0.92777" />
+      <inertia
+        ixx="0.0027392"
+        ixy="1.3667E-07"
+        ixz="-1.5309E-07"
+        iyy="0.0030619"
+        iyz="3.6492E-05"
+        izz="0.0053255" />
+    </inertial>
+    <visual>
+      <origin
+        xyz="0 0 0"
+        rpy="0 0 0" />
+      <geometry>
+        <mesh
+          filename="package://elfin_description/meshes/elfin10_l/elfin_base.STL" />
+      </geometry>
+      <material
+        name="">
+        <color
+          rgba="0.75294 0.75294 0.75294 1" />
+      </material>
+    </visual>
+    <collision>
+      <origin
+        xyz="0 0 0"
+        rpy="0 0 0" />
+      <geometry>
+        <mesh
+          filename="package://elfin_description/meshes/elfin10_l/elfin_base.STL" />
       </geometry>
     </collision>
@@ -68,37 +68,37 @@
     <inertial>
       <origin
-        xyz="-0.0040174 0.2265 4.5331E-06"
-        rpy="0 0 0" />
-      <mass
-        value="9.7894" />
-      <inertia
-        ixx="0.07916"
-        ixy="0.0021604"
-        ixz="4.5316E-06"
-        iyy="0.060146"
-        iyz="-5.7743E-06"
-        izz="0.088867" />
-    </inertial>
-    <visual>
-      <origin
-        xyz="0 0 0"
-        rpy="0 0 0" />
-      <geometry>
-        <mesh
-          filename="package://elfin_description/meshes/elfin15/elfin_link1.STL" />
-      </geometry>
-      <material
-        name="">
-        <color
-          rgba="0.79216 0.81961 0.93333 1" />
-      </material>
-    </visual>
-    <collision>
-      <origin
-        xyz="0 0 0"
-        rpy="0 0 0" />
-      <geometry>
-        <mesh
-          filename="package://elfin_description/meshes/elfin15/elfin_link1.STL" />
+        xyz="-0.027642 0.13484 1.9044E-05"
+        rpy="0 0 0" />
+      <mass
+        value="4.8966" />
+      <inertia
+        ixx="0.01645"
+        ixy="0.00098755"
+        ixz="-1.2324E-05"
+        iyy="0.014197"
+        iyz="-4.9714E-07"
+        izz="0.015841" />
+    </inertial>
+    <visual>
+      <origin
+        xyz="0 0 0"
+        rpy="0 0 0" />
+      <geometry>
+        <mesh
+          filename="package://elfin_description/meshes/elfin10_l/elfin_link1.STL" />
+      </geometry>
+      <material
+        name="">
+        <color
+          rgba="0.75294 0.75294 0.75294 1" />
+      </material>
+    </visual>
+    <collision>
+      <origin
+        xyz="0 0 0"
+        rpy="0 0 0" />
+      <geometry>
+        <mesh
+          filename="package://elfin_description/meshes/elfin10_l/elfin_link1.STL" />
       </geometry>
     </collision>
@@ -108,5 +108,5 @@
     type="revolute">
     <origin
-      xyz="0 0 0"
+      xyz="0 0 0.056998"
       rpy="1.5708 0 0" />
     <parent
@@ -126,37 +126,37 @@
     <inertial>
       <origin
-        xyz="-0.035073 0.29215 1.7591E-05"
-        rpy="0 0 0" />
-      <mass
-        value="9.5865" />
-      <inertia
-        ixx="0.59803"
-        ixy="-0.031615"
-        ixz="4.8599E-06"
-        iyy="0.022645"
-        iyz="-4.8185E-05"
-        izz="0.59118" />
-    </inertial>
-    <visual>
-      <origin
-        xyz="0 0 0"
-        rpy="0 0 0" />
-      <geometry>
-        <mesh
-          filename="package://elfin_description/meshes/elfin15/elfin_link2.STL" />
-      </geometry>
-      <material
-        name="">
-        <color
-          rgba="0.8902 0.8902 0.9098 1" />
-      </material>
-    </visual>
-    <collision>
-      <origin
-        xyz="0 0 0"
-        rpy="0 0 0" />
-      <geometry>
-        <mesh
-          filename="package://elfin_description/meshes/elfin15/elfin_link2.STL" />
+        xyz="-0.042656 0.26961 1.5893E-05"
+        rpy="0 0 0" />
+      <mass
+        value="2.4435" />
+      <inertia
+        ixx="0.091287"
+        ixy="-0.0033486"
+        ixz="2.0759E-06"
+        iyy="0.0058345"
+        iyz="-6.0394E-06"
+        izz="0.089301" />
+    </inertial>
+    <visual>
+      <origin
+        xyz="0 0 0"
+        rpy="0 0 0" />
+      <geometry>
+        <mesh
+          filename="package://elfin_description/meshes/elfin10_l/elfin_link2.STL" />
+      </geometry>
+      <material
+        name="">
+        <color
+          rgba="0.75294 0.75294 0.75294 1" />
+      </material>
+    </visual>
+    <collision>
+      <origin
+        xyz="0 0 0"
+        rpy="0 0 0" />
+      <geometry>
+        <mesh
+          filename="package://elfin_description/meshes/elfin10_l/elfin_link2.STL" />
       </geometry>
     </collision>
@@ -166,5 +166,5 @@
     type="revolute">
     <origin
-      xyz="-0.121 0.262 0"
+      xyz="-0.1025 0.202 0"
       rpy="0 0 0" />
     <parent
@@ -184,37 +184,37 @@
     <inertial>
       <origin
-        xyz="-0.0049696 -0.035269 2.0786E-06"
-        rpy="0 0 0" />
-      <mass
-        value="2.9386" />
-      <inertia
-        ixx="0.011876"
-        ixy="0.00059921"
-        ixz="1.0886E-07"
-        iyy="0.0075913"
-        iyz="4.8168E-07"
-        izz="0.013762" />
-    </inertial>
-    <visual>
-      <origin
-        xyz="0 0 0"
-        rpy="0 0 0" />
-      <geometry>
-        <mesh
-          filename="package://elfin_description/meshes/elfin15/elfin_link3.STL" />
-      </geometry>
-      <material
-        name="">
-        <color
-          rgba="1 1 1 1" />
-      </material>
-    </visual>
-    <collision>
-      <origin
-        xyz="0 0 0"
-        rpy="0 0 0" />
-      <geometry>
-        <mesh
-          filename="package://elfin_description/meshes/elfin15/elfin_link3.STL" />
+        xyz="-0.020704 -0.051289 2.5325E-05"
+        rpy="0 0 0" />
+      <mass
+        value="2.4293" />
+      <inertia
+        ixx="0.0049324"
+        ixy="0.00030979"
+        ixz="-4.991E-06"
+        iyy="0.0043065"
+        iyz="-1.2153E-06"
+        izz="0.0046452" />
+    </inertial>
+    <visual>
+      <origin
+        xyz="0 0 0"
+        rpy="0 0 0" />
+      <geometry>
+        <mesh
+          filename="package://elfin_description/meshes/elfin10_l/elfin_link3.STL" />
+      </geometry>
+      <material
+        name="">
+        <color
+          rgba="0.75294 0.75294 0.75294 1" />
+      </material>
+    </visual>
+    <collision>
+      <origin
+        xyz="0 0 0"
+        rpy="0 0 0" />
+      <geometry>
+        <mesh
+          filename="package://elfin_description/meshes/elfin10_l/elfin_link3.STL" />
       </geometry>
     </collision>
@@ -224,6 +224,6 @@
     type="revolute">
     <origin
-      xyz="0.121 0.73 0"
-      rpy="3.1416 0 0" />
+      xyz="0.1025 0.6 0"
+      rpy="-3.1416 0 0" />
     <parent
       link="elfin_link2" />
@@ -242,37 +242,37 @@
     <inertial>
       <origin
-        xyz="-0.064982 0.17333 3.5794E-05"
-        rpy="0 0 0" />
-      <mass
-        value="2.8258" />
-      <inertia
-        ixx="0.055923"
-        ixy="0.01272"
-        ixz="3.6239E-06"
-        iyy="0.0079448"
-        iyz="-1.9213E-05"
-        izz="0.060085" />
-    </inertial>
-    <visual>
-      <origin
-        xyz="0 0 0"
-        rpy="0 0 0" />
-      <geometry>
-        <mesh
-          filename="package://elfin_description/meshes/elfin15/elfin_link4.STL" />
-      </geometry>
-      <material
-        name="">
-        <color
-          rgba="0.79216 0.81961 0.93333 1" />
-      </material>
-    </visual>
-    <collision>
-      <origin
-        xyz="0 0 0"
-        rpy="0 0 0" />
-      <geometry>
-        <mesh
-          filename="package://elfin_description/meshes/elfin15/elfin_link4.STL" />
+        xyz="-0.066257 0.23401 1.1858E-05"
+        rpy="0 0 0" />
+      <mass
+        value="1.1159" />
+      <inertia
+        ixx="0.031789"
+        ixy="0.005014"
+        ixz="3.5796E-07"
+        iyy="0.0030538"
+        iyz="-5.4746E-06"
+        izz="0.032797" />
+    </inertial>
+    <visual>
+      <origin
+        xyz="0 0 0"
+        rpy="0 0 0" />
+      <geometry>
+        <mesh
+          filename="package://elfin_description/meshes/elfin10_l/elfin_link4.STL" />
+      </geometry>
+      <material
+        name="">
+        <color
+          rgba="0.75294 0.75294 0.75294 1" />
+      </material>
+    </visual>
+    <collision>
+      <origin
+        xyz="0 0 0"
+        rpy="0 0 0" />
+      <geometry>
+        <mesh
+          filename="package://elfin_description/meshes/elfin10_l/elfin_link4.STL" />
       </geometry>
     </collision>
@@ -300,37 +300,37 @@
     <inertial>
       <origin
-        xyz="-0.002491 -0.025023 -6.7752E-06"
-        rpy="0 0 0" />
-      <mass
-        value="1.2566" />
-      <inertia
-        ixx="0.0027306"
-        ixy="9.9756E-05"
-        ixz="4.9287E-07"
-        iyy="0.0020256"
-        iyz="-2.707E-07"
-        izz="0.0034996" />
-    </inertial>
-    <visual>
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
Commit message: update model and urdf

File: elfin_description/urdf/elfin10_l.urdf.xacro (robot description, xacro)
@@ -4,4 +4,5 @@
   <xacro:include filename="$(find elfin_description)/urdf/elfin_robot.gazebo" />
   <xacro:include filename="$(find elfin_description)/urdf/elfin_transmission.xacro" />
+  <xacro:property name="coef" value="0.000000001"/>
   <link name="world" />
   <joint name="world_base" type="fixed">
@@ -18,5 +19,5 @@
     <origin
       xyz="0 0 0"
-      rpy="0 0 1.5708" />
+      rpy="1.570797 ${1.570797*2} ${1.570797*2}" />
     <parent
       link="elfin_base_link" />
@@ -27,16 +28,16 @@
     name="elfin_base">
     <inertial>
-      <origin
-        xyz="3.0613E-07 0.0023359 0.025589"
-        rpy="0 0 0" />
-      <mass
-        value="0.92777" />
-      <inertia
-        ixx="0.0027392"
-        ixy="1.3667E-07"
-        ixz="-1.5309E-07"
-        iyy="0.0030619"
-        iyz="3.6492E-05"
-        izz="0.0053255" />
+        <origin
+        xyz="0.00032861 -0.02554 -0.00034505"
+        rpy="0 0 0" />
+      <mass
+        value="4.1802" />
+      <inertia
+        ixx="0.0075485"
+        ixy="1.0006E-05"
+        ixz="-4.3994E-05"
+        iyy="0.014632"
+        iyz="-0.00010482"
+        izz="0.0084243" />
     </inertial>
     <visual>
@@ -51,5 +52,5 @@
         name="">
         <color
-          rgba="0.75294 0.75294 0.75294 1" />
+          rgba="0.86667 0.86667 0.8902 1" />
       </material>
     </visual>
@@ -67,16 +68,16 @@
     name="elfin_link1">
     <inertial>
-      <origin
-        xyz="-0.027642 0.13484 1.9044E-05"
-        rpy="0 0 0" />
-      <mass
-        value="4.8966" />
-      <inertia
-        ixx="0.01645"
-        ixy="0.00098755"
-        ixz="-1.2324E-05"
-        iyy="0.014197"
-        iyz="-4.9714E-07"
-        izz="0.015841" />
+        <origin
+        xyz="2.6857E-05 -0.029266 0.1919"
+        rpy="0 0 0" />
+      <mass
+        value="16.609" />
+      <inertia
+        ixx="0.034331"
+        ixy="-3.4482E-05"
+        ixz="-2.9633E-05"
+        iyy="0.045424"
+        iyz="0.0022102"
+        izz="0.039605" />
     </inertial>
     <visual>
@@ -91,5 +92,5 @@
         name="">
         <color
-          rgba="0.75294 0.75294 0.75294 1" />
+          rgba="1 1 1 1" />
       </material>
     </visual>
@@ -108,5 +109,5 @@
     type="revolute">
     <origin
-      xyz="0 0 0.056998"
+      xyz="0 0 0"
       rpy="1.5708 0 0" />
     <parent
@@ -115,5 +116,5 @@
       link="elfin_link1" />
     <axis
-      xyz="0 1 0" />
+      xyz="0 0 1" />
     <limit
       lower="-3.14"
@@ -125,16 +126,16 @@
     name="elfin_link2">
     <inertial>
-      <origin
-        xyz="-0.042656 0.26961 1.5893E-05"
-        rpy="0 0 0" />
-      <mass
-        value="2.4435" />
-      <inertia
-        ixx="0.091287"
-        ixy="-0.0033486"
-        ixz="2.0759E-06"
-        iyy="0.0058345"
-        iyz="-6.0394E-06"
-        izz="0.089301" />
+         <origin
+        xyz="1.4387E-05 0.26969 0.14233"
+        rpy="0 0 0" />
+      <mass
+        value="8.7235" />
+      <inertia
+        ixx="0.24536"
+        ixy="-2.4916E-05"
+        ixz="-5.9253E-06"
+        iyy="0.015887"
+        iyz="0.0081398"
+        izz="0.25053" />
     </inertial>
     <visual>
@@ -149,5 +150,5 @@
         name="">
         <color
-          rgba="0.75294 0.75294 0.75294 1" />
+          rgba="1 1 1 1" />
       </material>
     </visual>
@@ -166,6 +167,6 @@
     type="revolute">
     <origin
-      xyz="-0.1025 0.202 0"
-      rpy="0 0 0" />
+      xyz="0 0 0.26"
+      rpy="1.5708 0 0" />
     <parent
       link="elfin_link1" />
@@ -173,5 +174,5 @@
       link="elfin_link2" />
     <axis
-      xyz="-1 0 0" />
+      xyz="0 0 1" />
     <limit
       lower="-2.35"
@@ -183,16 +184,16 @@
     name="elfin_link3">
     <inertial>
-      <origin
-        xyz="-0.020704 -0.051289 2.5325E-05"
-        rpy="0 0 0" />
-      <mass
-        value="2.4293" />
-      <inertia
-        ixx="0.0049324"
-        ixy="0.00030979"
-        ixz="-4.991E-06"
-        iyy="0.0043065"
-        iyz="-1.2153E-06"
-        izz="0.0046452" />
+        <origin
+        xyz="0.053847 -1.0028E-05 -0.023648"
+        rpy="0 0 0" />
+      <mass
+        value="8.28817" />
+      <inertia
+        ixx="0.013498"
+        ixy="5.7296E-06"
+        ixz="-0.00075857"
+        iyy="0.011546"
+        iyz="4.255E-06"
+        izz="0.015027" />
     </inertial>
     <visual>
@@ -207,5 +208,5 @@
         name="">
         <color
-          rgba="0.75294 0.75294 0.75294 1" />
+          rgba="1 1 1 1" />
       </material>
     </visual>
@@ -224,6 +225,6 @@
     type="revolute">
     <origin
-      xyz="0.1025 0.6 0"
-      rpy="-3.1416 0 0" />
+      xyz="0 0.6 0"
+      rpy="3.1416 0 1.5708" />
     <parent
       link="elfin_link2" />
@@ -231,5 +232,5 @@
       link="elfin_link3" />
     <axis
-      xyz="1 0 0" />
+      xyz="0 0 1" />
     <limit
       lower="-2.61"
@@ -241,16 +242,16 @@
     name="elfin_link4">
     <inertial>
-      <origin
-        xyz="-0.066257 0.23401 1.1858E-05"
-        rpy="0 0 0" />
-      <mass
-        value="1.1159" />
-      <inertia
-        ixx="0.031789"
-        ixy="0.005014"
-        ixz="3.5796E-07"
-        iyy="0.0030538"
-        iyz="-5.4746E-06"
-        izz="0.032797" />
+         <origin
+        xyz="2.0335E-05 -0.067673 0.38361"
+        rpy="0 0 0" />
+      <mass
+        value="4.09857" />
+      <inertia
+        ixx="0.091784"
+        ixy="1.3519E-07"
+        ixz="-1.4394E-05"
+        iyy="0.08887"
+        iyz="0.014085"
+        izz="0.0084778" />
     </inertial>
     <visual>
@@ -265,5 +266,5 @@
         name="">
         <color
-          rgba="0.75294 0.75294 0.75294 1" />
+          rgba="0.792156862745098 0.819607843137255 0.933333333333333 1" />
       </material>
     </visual>
@@ -282,6 +283,6 @@
     type="revolute">
     <origin
-      xyz="0 -0.147 0"
-      rpy="-3.1416 0 0" />
+      xyz="0 0 0"
+      rpy="1.5708 0 1.5708" />
     <parent
       link="elfin_link3" />
@@ -289,5 +290,5 @@
       link="elfin_link4" />
     <axis
-      xyz="0 1 0" />
+      xyz="0 0 1" />
     <limit
       lower="-3.14"
@@ -299,16 +300,16 @@
     name="elfin_link5">
     <inertial>
-      <origin
-        xyz="-0.016508 -0.036734 -5.1662E-06"
-        rpy="0 0 0" />
-      <mass
-        value="1.0836" />
-      <inertia
-        ixx="0.0012538"
-        ixy="8.3769E-05"
-        ixz="4.7317E-07"
-        iyy="0.0011133"
-        iyz="-2.0722E-07"
-        izz="0.0013201" />
+        <origin
+        xyz="-2.5145E-05 -0.039561 -0.01936"
+        rpy="0 0 0" />
+      <mass
+        value="3.74304" />
+      <inertia
+        ixx="0.0027397"
+        ixy="-7.4484E-06"
+        ixz="1.5721E-05"
+        iyy="0.0030296"
+        iyz="0.00020143"
+        izz="0.0033511" />
     </inertial>
     <visual>
@@ -323,5 +324,5 @@
         name="">
         <color
-          rgba="0.75294 0.75294 0.75294 1" />
+          rgba="1 1 1 1" />
       </material>
     </visual>
@@ -340,6 +341,6 @@
     type="revolute">
     <origin
-      xyz="0 0.553 0"
-      rpy="3.1416 0 0" />
+      xyz="0 0 0.7"
+      rpy="-1.5708 0 0" />
     <parent
       link="elfin_link4" />
@@ -347,5 +348,5 @@
       link="elfin_link5" />
     <axis
-      xyz="1 0 0" />
+      xyz="0 0 1" />
     <limit
       lower="-2.56"
@@ -357,16 +358,16 @@
     name="elfin_link6">
     <inertial>
-      <origin
-        xyz="-0.007186 -0.015033 2.0521E-05"
-        rpy="0 0 0" />
-      <mass
-        value="0.11713" />
-      <inertia
-        ixx="8.0778E-05"
-        ixy="-2.1206E-06"
-        ixz="-1.0023E-07"
-        iyy="0.00013969"
-        iyz="-3.1713E-08"
-        izz="8.3118E-05" />
+        <origin
+        xyz="0.00091682 -0.0048568 0.14017"
+        rpy="0 0 0" />
+      <mass
+        value="0.82406" />
+      <inertia
+        ixx="0.00032663"
+        ixy="-1.3657E-07"
+        ixz="-2.3073E-09"
+        iyy="0.00032085"
+        iyz="-5.7935E-06"
+        izz="0.00056343" />
     </inertial>
     <visual>
@@ -381,5 +382,5 @@
         name="">
         <color
-          rgba="0.75294 0.75294 0.75294 1" />
+          rgba="1 1 1 1" />
       </material>
     </visual>
@@ -398,6 +399,6 @@
     type="revolute">
     <origin
-      xyz="0 -0.1595 0"
-      rpy="-3.1416 0 0" />
+      xyz="0 0 0"
+      rpy="1.5708 0 0" />
     <parent
       link="elfin_link5" />
@@ -405,5 +406,5 @@
       link="elfin_link6" />
     <axis
-      xyz="0 1 0" />
+      xyz="0 0 1" />
     <limit
       lower="-3.14"
@@ -412,11 +413,11 @@
       velocity="1.57" />
   </joint>
-  <link name="elfin_end_link" />
+  <link name="elfin_end_link"/>
   <joint
     name="elfin_end_joint"
     type="fixed">
     <origin
-      xyz="0 0.0095 0"
-      rpy="-1.5708 -1.5708 0" />
+      xyz="0 0 0.168"
+      rpy="0 0 0" />
     <parent
       link="elfin_link6" />
@@ -426,5 +427,5 @@
       xyz="0 0 0" />
   </joint>
-  <link name="elfin_dummy_gripper"/>
+ <link name="elfin_dummy_gripper"/>
   <joint name="elfin_dummy_joint" type="fixed">
     <origin
