Commit message: update
update model

File: elfin_description/urdf/elfin5_l.urdf.xacro (robot description, xacro)
@@ -28,37 +28,37 @@
     <inertial>
       <origin
-        xyz="-0.0007634 5.6362E-06 0.030441"
-        rpy="0 0 0" />
-      <mass
-        value="0.97022" />
-      <inertia
-        ixx="0.0015769"
-        ixy="1.2223E-07"
-        ixz="-2.1696E-05"
-        iyy="0.0014456"
-        iyz="-6.1863E-08"
-        izz="0.0023657" />
-    </inertial>
-    <visual>
-      <origin
-        xyz="0 0 0"
-        rpy="0 0 0" />
-      <geometry>
-        <mesh
-          filename="package://elfin_description/meshes/elfin5_l/elfin_base_link.STL" />
-      </geometry>
-      <material
-        name="">
-        <color
-          rgba="0.75294 0.75294 0.75294 1" />
-      </material>
-    </visual>
-    <collision>
-      <origin
-        xyz="0 0 0"
-        rpy="0 0 0" />
-      <geometry>
-        <mesh
-          filename="package://elfin_description/meshes/elfin5_l/elfin_base_link.STL" />
+        xyz="-0.00199130179727394 7.44168336203446E-06 0.0272977448147404"
+        rpy="0 0 0" />
+      <mass
+        value="0.546250568289568" />
+      <inertia
+        ixx="0.00118732326275469"
+        ixy="5.36844840925411E-07"
+        ixz="-2.09426769103823E-05"
+        iyy="0.00103230683074767"
+        iyz="-1.04918150299868E-07"
+        izz="0.00193030289476119" />
+    </inertial>
+    <visual>
+      <origin
+        xyz="0 0 0"
+        rpy="0 0 0" />
+      <geometry>
+        <mesh
+          filename="package://elfin_description/meshes/elfin5_l/elfin_base.STL" />
+      </geometry>
+      <material
+        name="">
+        <color
+          rgba="0.792156862745098 0.819607843137255 0.933333333333333 1" />
+      </material>
+    </visual>
+    <collision>
+      <origin
+        xyz="0 0 0"
+        rpy="0 0 0" />
+      <geometry>
+        <mesh
+          filename="package://elfin_description/meshes/elfin5_l/elfin_base.STL" />
       </geometry>
     </collision>
@@ -68,15 +68,15 @@
     <inertial>
       <origin
-        xyz="3.3881E-06 -0.0059071 0.10092"
-        rpy="0 0 0" />
-      <mass
-        value="3.1643" />
-      <inertia
-        ixx="0.012965"
-        ixy="6.1671E-08"
-        ixz="4.3957E-07"
-        iyy="0.012144"
-        iyz="0.0023647"
-        izz="0.0069485" />
+        xyz="3.55428747498904E-05 -0.0238032507595431 -0.056664005378111"
+        rpy="0 0 0" />
+      <mass
+        value="1.71757344675846" />
+      <inertia
+        ixx="0.00313309686683817"
+        ixy="-6.81025650006338E-07"
+        ixz="-2.50470833748591E-06"
+        iyy="0.00372508389579096"
+        iyz="0.000325673248643593"
+        izz="0.00319411847606861" />
     </inertial>
     <visual>
@@ -91,5 +91,5 @@
         name="">
         <color
-          rgba="0.75294 0.75294 0.75294 1" />
+          rgba="0.792156862745098 0.819607843137255 0.933333333333333 1" />
       </material>
     </visual>
@@ -108,5 +108,5 @@
     type="revolute">
     <origin
-      xyz="0 0 0.082"
+      xyz="0 0 0.22"
       rpy="0 0 0" />
     <parent
@@ -119,5 +119,5 @@
       lower="-3.14"
       upper="3.14"
-      effort="420"
+      effort="104"
       velocity="1.57" />
   </joint>
@@ -126,15 +126,15 @@
     <inertial>
       <origin
-        xyz="-1.114E-05 -0.049377 0.19342"
-        rpy="0 0 0" />
-      <mass
-        value="3.1869" />
-      <inertia
-        ixx="0.073265"
-        ixy="5.1353E-07"
-        ixz="-2.6175E-06"
-        iyy="0.073984"
-        iyz="-0.0020394"
-        izz="0.0031464" />
+        xyz="-8.02320899791198E-06 0.194762833402907 0.128888916941187"
+        rpy="0 0 0" />
+      <mass
+        value="1.10522962809227" />
+      <inertia
+        ixx="0.0225843178593198"
+        ixy="-7.27982747203185E-07"
+        ixz="-1.78485875318381E-07"
+        iyy="0.00152004282471311"
+        iyz="0.000623589021520354"
+        izz="0.0230428803086098" />
     </inertial>
     <visual>
@@ -149,5 +149,5 @@
         name="">
         <color
-          rgba="0.75294 0.75294 0.75294 1" />
+          rgba="0.792156862745098 0.819607843137255 0.933333333333333 1" />
       </material>
     </visual>
@@ -166,6 +166,6 @@
     type="revolute">
     <origin
-      xyz="0 -0.07785 0.138"
-      rpy="0 0 0" />
+      xyz="0 0 0"
+      rpy="1.5708 0 0" />
     <parent
       link="elfin_link1" />
@@ -173,10 +173,10 @@
       link="elfin_link2" />
     <axis
-      xyz="0 -1 0" />
-    <limit
+      xyz="0 0 1" />
+     <limit
       lower="-2.35"
       upper="2.35"
-      effort="420"
-      velocity="1.57" />
+      effort="104"
+      velocity="1.27" />
   </joint>
   <link
@@ -184,15 +184,15 @@
     <inertial>
       <origin
-        xyz="9.3762E-06 0.066365 0.030316"
-        rpy="0 0 0" />
-      <mass
-        value="1.9252" />
-      <inertia
-        ixx="0.0058726"
-        ixy="7.1997E-07"
-        ixz="-2.9335E-07"
-        iyy="0.0051729"
-        iyz="-0.0011237"
-        izz="0.0031696" />
+        xyz="0.0461694549854045 1.67843463302067E-05 -0.0210719533256843"
+        rpy="0 0 0" />
+      <mass
+        value="1.07590672952063" />
+      <inertia
+        ixx="0.00137807691049161"
+        ixy="-3.57302576480749E-07"
+        ixz="-0.00013179565326652"
+        iyy="0.00135308160804782"
+        iyz="9.02259193989242E-07"
+        izz="0.00154416453671479" />
     </inertial>
     <visual>
@@ -207,5 +207,5 @@
         name="">
         <color
-          rgba="0.75294 0.75294 0.75294 1" />
+          rgba="0.792156862745098 0.819607843137255 0.933333333333333 1" />
       </material>
     </visual>
@@ -224,6 +224,6 @@
     type="revolute">
     <origin
-      xyz="0 0.00585 0.455"
-      rpy="0 0 0" />
+      xyz="0 0.455 0"
+      rpy="-3.1416 0 1.5708" />
     <parent
       link="elfin_link2" />
@@ -231,177 +231,61 @@
       link="elfin_link3" />
     <axis
-      xyz="0 1 0" />
+      xyz="0 0 1" />
     <limit
       lower="-2.61"
       upper="2.61"
-      effort="200"
-      velocity="1.57" />
-  </joint>
-  <link
-    name="elfin_link4">
-    <inertial>
-      <origin
-        xyz="-2.4659E-05 -0.042655 0.16376"
-        rpy="0 0 0" />
-      <mass
-        value="1.94" />
-      <inertia
-        ixx="0.025102"
-        ixy="-2.7421E-06"
-        ixz="8.4771E-06"
-        iyy="0.022005"
-        iyz="0.0071908"
-        izz="0.0050335" />
-    </inertial>
-    <visual>
-      <origin
-        xyz="0 0 0"
-        rpy="0 0 0" />
-      <geometry>
-        <mesh
-          filename="package://elfin_description/meshes/elfin5_l/elfin_link4.STL" />
-      </geometry>
-      <material
-        name="">
-        <color
-          rgba="0.75294 0.75294 0.75294 1" />
-      </material>
-    </visual>
-    <collision>
-      <origin
-        xyz="0 0 0"
-        rpy="0 0 0" />
-      <geometry>
-        <mesh
-          filename="package://elfin_description/meshes/elfin5_l/elfin_link4.STL" />
-      </geometry>
-    </collision>
-  </link>
-  <joint
-    name="elfin_joint4"
-    type="revolute">
-    <origin
-      xyz="0 0.072 0.117"
-      rpy="0 0 0" />
-    <parent
-      link="elfin_link3" />
-    <child
-      link="elfin_link4" />
-    <axis
-      xyz="0 0 1" />
-    <limit
-      lower="-3.14"
-      upper="3.14"
-      effort="200"
-      velocity="1.57" />
-  </joint>
-  <link
-    name="elfin_link5">
-    <inertial>
-      <origin
-        xyz="-4.9859E-07 0.055949 0.022517"
-        rpy="0 0 0" />
-      <mass
-        value="0.9902" />
-      <inertia
-        ixx="0.0019311"
-        ixy="1.0751E-07"
-        ixz="-3.2968E-08"
-        iyy="0.0016081"
-        iyz="-0.00037481"
-        izz="0.0010972" />
-    </inertial>
-    <visual>
-      <origin
-        xyz="0 0 0"
-        rpy="0 0 0" />
-      <geometry>
-        <mesh
-          filename="package://elfin_description/meshes/elfin5_l/elfin_link5.STL" />
-      </geometry>
-      <material
-        name="">
-        <color
-          rgba="0.75294 0.75294 0.75294 1" />
-      </material>
-    </visual>
-    <collision>
-      <origin
-        xyz="0 0 0"
-        rpy="0 0 0" />
-      <geometry>
-        <mesh
-          filename="package://elfin_description/meshes/elfin5_l/elfin_link5.STL" />
-      </geometry>
-    </collision>
-  </link>
-  <joint
-    name="elfin_joint5"
-    type="revolute">
-    <origin
-      xyz="0 -0.060249 0.378"
-      rpy="0 0 0" />
-    <parent
-      link="elfin_link4" />
-    <child
-      link="elfin_link5" />
-    <axis
-      xyz="0 1 0" />
-    <limit
-      lower="-2.56"
-      upper="2.56"
       effort="69"
       velocity="1.57" />
   </joint>
   <link
-    name="elfin_link6">
-    <inertial>
-      <origin
-        xyz="0.00019949 -0.0025865 0.030984"
-        rpy="0 0 0" />
-      <mass
-        value="0.22732" />
-      <inertia
-        ixx="0.000125"
-        ixy="-2.5767E-07"
-        ixz="7.1113E-09"
-        iyy="0.00013055"
-        iyz="1.8454E-07"
-        izz="0.00020378" />
-    </inertial>
-    <visual>
-      <origin
-        xyz="0 0 0"
-        rpy="0 0 0" />
-      <geometry>
-        <mesh
-          filename="package://elfin_description/meshes/elfin5_l/elfin_link6.STL" />
-      </geometry>
-      <material
-        name="">
-        <color
-          rgba="0.75294 0.75294 0.75294 1" />
-      </material>
-    </visual>
-    <collision>
-      <origin
-        xyz="0 0 0"
-        rpy="0 0 0" />
-      <geometry>
-        <mesh
-          filename="package://elfin_description/meshes/elfin5_l/elfin_link6.STL" />
-      </geometry>
-    </collision>
-  </link>
-  <joint
-    name="elfin_joint6"
-    type="revolute">
-    <origin
-      xyz="0 0.060249 0.09175"
-      rpy="0 0 0" />
-    <parent
-      link="elfin_link5" />
-    <child
-      link="elfin_link6" />
+    name="elfin_link4">
+    <inertial>
+      <origin
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