Commit message: update elfin5-l(1316mm)  moveit_package/urdf/model_description,add elfin5_l ikFastPlugin

File: elfin_description/urdf/elfin5_l.urdf.xacro (robot description, xacro)
@@ -18,5 +18,5 @@
     <origin
       xyz="0 0 0"
-      rpy="0 0 1.5708" />
+      rpy="0 0 0" />
     <parent
       link="elfin_base_link" />
@@ -28,37 +28,37 @@
     <inertial>
       <origin
-        xyz="0.00022093 0.0013404 0.025529"
-        rpy="0 0 0" />
-      <mass
-        value="0.68795" />
-      <inertia
-        ixx="0.0012704"
-        ixy="6.1256E-06"
-        ixz="1.9788E-06"
-        iyy="0.0013413"
-        iyz="1.2007E-05"
-        izz="0.0022564" />
-    </inertial>
-    <visual>
-      <origin
-        xyz="0 0 0"
-        rpy="0 0 0" />
-      <geometry>
-        <mesh
-          filename="package://elfin_description/meshes/elfin5_l/elfin_base.STL" />
-      </geometry>
-      <material
-        name="">
-        <color
-          rgba="0.79216 0.81961 0.92941 1" />
-      </material>
-    </visual>
-    <collision>
-      <origin
-        xyz="0 0 0"
-        rpy="0 0 0" />
-      <geometry>
-        <mesh
-          filename="package://elfin_description/meshes/elfin5_l/elfin_base.STL" />
+        xyz="-0.0007634 5.6362E-06 0.030441"
+        rpy="0 0 0" />
+      <mass
+        value="0.97022" />
+      <inertia
+        ixx="0.0015769"
+        ixy="1.2223E-07"
+        ixz="-2.1696E-05"
+        iyy="0.0014456"
+        iyz="-6.1863E-08"
+        izz="0.0023657" />
+    </inertial>
+    <visual>
+      <origin
+        xyz="0 0 0"
+        rpy="0 0 0" />
+      <geometry>
+        <mesh
+          filename="package://elfin_description/meshes/elfin5_l/elfin_base_link.STL" />
+      </geometry>
+      <material
+        name="">
+        <color
+          rgba="0.75294 0.75294 0.75294 1" />
+      </material>
+    </visual>
+    <collision>
+      <origin
+        xyz="0 0 0"
+        rpy="0 0 0" />
+      <geometry>
+        <mesh
+          filename="package://elfin_description/meshes/elfin5_l/elfin_base_link.STL" />
       </geometry>
     </collision>
@@ -68,15 +68,15 @@
     <inertial>
       <origin
-        xyz="-0.021818 0.13889 0.000013458"
-        rpy="0 0 0" />
-      <mass
-        value="2.5856" />
-      <inertia
-        ixx="0.012636"
-        ixy="0.0034176"
-        ixz="-1.9559E-06"
-        iyy="0.0066118"
-        iyz="-1.7982E-06"
-        izz="0.014362" />
+        xyz="3.3881E-06 -0.0059071 0.10092"
+        rpy="0 0 0" />
+      <mass
+        value="3.1643" />
+      <inertia
+        ixx="0.012965"
+        ixy="6.1671E-08"
+        ixz="4.3957E-07"
+        iyy="0.012144"
+        iyz="0.0023647"
+        izz="0.0069485" />
     </inertial>
     <visual>
@@ -91,5 +91,5 @@
         name="">
         <color
-          rgba="0.77255 0.75294 0.73333 1" />
+          rgba="0.75294 0.75294 0.75294 1" />
       </material>
     </visual>
@@ -108,6 +108,6 @@
     type="revolute">
     <origin
-      xyz="0 0 0.03"
-      rpy="1.5708 0 0" />
+      xyz="0 0 0.082"
+      rpy="0 0 0" />
     <parent
       link="elfin_base" />
@@ -115,5 +115,5 @@
       link="elfin_link1" />
     <axis
-      xyz="0 1 0" />
+      xyz="0 0 1" />
     <limit
       lower="-3.14"
@@ -126,15 +126,15 @@
     <inertial>
       <origin
-        xyz="-0.032497 0.30341 -7.6521E-05"
-        rpy="0 0 0" />
-      <mass
-        value="1.208607" />
-      <inertia
-        ixx="0.02975970"
-        ixy="-0.00126441"
-        ixz="-0.00000024"
-        iyy="0.00168156"
-        iyz="-0.0000021"
-        izz="0.02944694" />
+        xyz="-1.114E-05 -0.049377 0.19342"
+        rpy="0 0 0" />
+      <mass
+        value="3.1869" />
+      <inertia
+        ixx="0.073265"
+        ixy="5.1353E-07"
+        ixz="-2.6175E-06"
+        iyy="0.073984"
+        iyz="-0.0020394"
+        izz="0.0031464" />
     </inertial>
     <visual>
@@ -149,5 +149,5 @@
         name="">
         <color
-          rgba="0.68627 0.68627 0.68627 1" />
+          rgba="0.75294 0.75294 0.75294 1" />
       </material>
     </visual>
@@ -166,5 +166,5 @@
     type="revolute">
     <origin
-      xyz="-0.087 0.19 0"
+      xyz="0 -0.07785 0.138"
       rpy="0 0 0" />
     <parent
@@ -173,5 +173,5 @@
       link="elfin_link2" />
     <axis
-      xyz="-1 0 0" />
+      xyz="0 -1 0" />
     <limit
       lower="-2.35"
@@ -184,15 +184,15 @@
     <inertial>
       <origin
-        xyz="0.067584 -0.041479 -1.1421E-05"
-        rpy="0 0 0" />
-      <mass
-        value="1.5324" />
-      <inertia
-        ixx="0.00514"
-        ixy="0.0014834"
-        ixz="-5.7782E-07"
-        iyy="0.0028926"
-        iyz="-3.0654E-07"
-        izz="0.0060883" />
+        xyz="9.3762E-06 0.066365 0.030316"
+        rpy="0 0 0" />
+      <mass
+        value="1.9252" />
+      <inertia
+        ixx="0.0058726"
+        ixy="7.1997E-07"
+        ixz="-2.9335E-07"
+        iyy="0.0051729"
+        iyz="-0.0011237"
+        izz="0.0031696" />
     </inertial>
     <visual>
@@ -207,5 +207,5 @@
         name="">
         <color
-          rgba="0.86667 0.86667 0.8902 1" />
+          rgba="0.75294 0.75294 0.75294 1" />
       </material>
     </visual>
@@ -224,6 +224,6 @@
     type="revolute">
     <origin
-      xyz="0 0.455 0"
-      rpy="-3.1416 0 0" />
+      xyz="0 0.00585 0.455"
+      rpy="0 0 0" />
     <parent
       link="elfin_link2" />
@@ -231,5 +231,5 @@
       link="elfin_link3" />
     <axis
-      xyz="1 0 0" />
+      xyz="0 1 0" />
     <limit
       lower="-2.61"
@@ -242,15 +242,15 @@
     <inertial>
       <origin
-        xyz="-0.017434 -0.33294 -0.00015134"
-        rpy="0 0 0" />
-      <mass
-        value="0.5" />
-      <inertia
-        ixx="0.00542441"
-        ixy="0.0020749"
-        ixz="1.0501E-05"
-        iyy="0.014338"
-        iyz="-0.00041574"
-        izz="0.00607489" />
+        xyz="-2.4659E-05 -0.042655 0.16376"
+        rpy="0 0 0" />
+      <mass
+        value="1.94" />
+      <inertia
+        ixx="0.025102"
+        ixy="-2.7421E-06"
+        ixz="8.4771E-06"
+        iyy="0.022005"
+        iyz="0.0071908"
+        izz="0.0050335" />
     </inertial>
     <visual>
@@ -265,5 +265,5 @@
         name="">
         <color
-          rgba="0.68627 0.68627 0.68627 1" />
+          rgba="0.75294 0.75294 0.75294 1" />
       </material>
     </visual>
@@ -282,6 +282,6 @@
     type="revolute">
     <origin
-      xyz="0.087 -0.1255 0"
-      rpy="3.1416 0 0" />
+      xyz="0 0.072 0.117"
+      rpy="0 0 0" />
     <parent
       link="elfin_link3" />
@@ -289,5 +289,5 @@
       link="elfin_link4" />
     <axis
-      xyz="0 1 0" />
+      xyz="0 0 1" />
     <limit
       lower="-3.14"
@@ -300,15 +300,15 @@
     <inertial>
       <origin
-        xyz="-0.015972 -0.036591 1.4235E-06"
-        rpy="0 0 0" />
-      <mass
-        value="0.81192" />
-      <inertia
-        ixx="0.0018901"
-        ixy="0.00056728"
-        ixz="-4.2025E-08"
-        iyy="0.0010231"
-        iyz="5.0791E-09"
-        izz="0.002299" />
+        xyz="-4.9859E-07 0.055949 0.022517"
+        rpy="0 0 0" />
+      <mass
+        value="0.9902" />
+      <inertia
+        ixx="0.0019311"
+        ixy="1.0751E-07"
+        ixz="-3.2968E-08"
+        iyy="0.0016081"
+        iyz="-0.00037481"
+        izz="0.0010972" />
     </inertial>
     <visual>
@@ -323,5 +323,5 @@
         name="">
         <color
-          rgba="0.79216 0.81961 0.93333 1" />
+          rgba="0.75294 0.75294 0.75294 1" />
       </material>
     </visual>
@@ -340,6 +340,6 @@
     type="revolute">
     <origin
-      xyz="0 0.3695 0"
-      rpy="-3.1416 0 0" />
+      xyz="0 -0.060249 0.378"
+      rpy="0 0 0" />
     <parent
       link="elfin_link4" />
@@ -347,5 +347,5 @@
       link="elfin_link5" />
     <axis
-      xyz="1 0 0" />
+      xyz="0 1 0" />
     <limit
       lower="-2.56"
@@ -358,15 +358,15 @@
     <inertial>
       <origin
-        xyz="-0.0072549 0.027062 3.208E-05"
-        rpy="0 0 0" />
-      <mass
-        value="0.11343" />
-      <inertia
-        ixx="7.4923E-05"
-        ixy="-2.3429E-06"
-        ixz="-1.8394E-07"
-        iyy="0.0001278"
-        iyz="-4.8092E-08"
-        izz="7.6653E-05" />
+        xyz="0.00019949 -0.0025865 0.030984"
+        rpy="0 0 0" />
+      <mass
+        value="0.22732" />
+      <inertia
+        ixx="0.000125"
+        ixy="-2.5767E-07"
+        ixz="7.1113E-09"
+        iyy="0.00013055"
+        iyz="1.8454E-07"
+        izz="0.00020378" />
     </inertial>
     <visual>
@@ -381,5 +381,5 @@
         name="">
         <color
-          rgba="0.77647 0.75686 0.73725 1" />
+          rgba="0.75294 0.75294 0.75294 1" />
       </material>
     </visual>
@@ -398,6 +398,6 @@
     type="revolute">
     <origin
-      xyz="0 -0.1065 0"
-      rpy="3.1416 0 0" />
+      xyz="0 0.060249 0.09175"
+      rpy="0 0 0" />
     <parent
       link="elfin_link5" />
@@ -405,5 +405,5 @@
       link="elfin_link6" />
     <axis
-      xyz="0 1 0" />
+      xyz="0 0 1" />
     <limit
       lower="-3.14"
@@ -412,11 +412,11 @@
       velocity="1.57" />
   </joint>
-  <link name="elfin_end_link" />
+  <link name="elfin_end_link"/>
   <joint
     name="elfin_end_joint"
     type="fixed">
     <origin
-      xyz="0 0.04 0"
-      rpy="1.5708 -1.5708 0" />
+      xyz="0.0 0.0 0.05425"
+      rpy="0 0 0" />
     <parent
       link="elfin_link6" />

Commit message: update model
update model

File: elfin_description/urdf/elfin5_l.urdf.xacro (robot description, xacro)
@@ -18,5 +18,5 @@
     <origin
       xyz="0 0 0"
-      rpy="0 0 1.5708" />
+      rpy="0 0 0" />
     <parent
       link="elfin_base_link" />
@@ -28,15 +28,15 @@
     <inertial>
       <origin
-        xyz="0.00022093 0.0013404 0.025529"
-        rpy="0 0 0" />
-      <mass
-        value="0.68795" />
-      <inertia
-        ixx="0.0012704"
-        ixy="6.1256E-06"
-        ixz="1.9788E-06"
-        iyy="0.0013413"
-        iyz="1.2007E-05"
-        izz="0.0022564" />
+        xyz="-0.00199130179727394 7.44168336203446E-06 0.0272977448147404"
+        rpy="0 0 0" />
+      <mass
+        value="0.546250568289568" />
+      <inertia
+        ixx="0.00118732326275469"
+        ixy="5.36844840925411E-07"
+        ixz="-2.09426769103823E-05"
+        iyy="0.00103230683074767"
+        iyz="-1.04918150299868E-07"
+        izz="0.00193030289476119" />
     </inertial>
     <visual>
@@ -51,5 +51,5 @@
         name="">
         <color
-          rgba="0.79216 0.81961 0.92941 1" />
+          rgba="0.792156862745098 0.819607843137255 0.933333333333333 1" />
       </material>
     </visual>
@@ -68,15 +68,15 @@
     <inertial>
       <origin
-        xyz="-0.021818 0.13889 0.000013458"
-        rpy="0 0 0" />
-      <mass
-        value="2.5856" />
-      <inertia
-        ixx="0.012636"
-        ixy="0.0034176"
-        ixz="-1.9559E-06"
-        iyy="0.0066118"
-        iyz="-1.7982E-06"
-        izz="0.014362" />
+        xyz="3.55428747498904E-05 -0.0238032507595431 -0.056664005378111"
+        rpy="0 0 0" />
+      <mass
+        value="1.71757344675846" />
+      <inertia
+        ixx="0.00313309686683817"
+        ixy="-6.81025650006338E-07"
+        ixz="-2.50470833748591E-06"
+        iyy="0.00372508389579096"
+        iyz="0.000325673248643593"
+        izz="0.00319411847606861" />
     </inertial>
     <visual>
@@ -91,5 +91,5 @@
         name="">
         <color
-          rgba="0.77255 0.75294 0.73333 1" />
+          rgba="0.792156862745098 0.819607843137255 0.933333333333333 1" />
       </material>
     </visual>
@@ -108,6 +108,6 @@
     type="revolute">
     <origin
-      xyz="0 0 0.03"
-      rpy="1.5708 0 0" />
+      xyz="0 0 0.22"
+      rpy="0 0 0" />
     <parent
       link="elfin_base" />
@@ -115,9 +115,9 @@
       link="elfin_link1" />
     <axis
-      xyz="0 1 0" />
+      xyz="0 0 1" />
     <limit
       lower="-3.14"
       upper="3.14"
-      effort="420"
+      effort="104"
       velocity="1.57" />
   </joint>
@@ -126,15 +126,15 @@
     <inertial>
       <origin
-        xyz="-0.032497 0.30341 -7.6521E-05"
-        rpy="0 0 0" />
-      <mass
-        value="1.208607" />
-      <inertia
-        ixx="0.02975970"
-        ixy="-0.00126441"
-        ixz="-0.00000024"
-        iyy="0.00168156"
-        iyz="-0.0000021"
-        izz="0.02944694" />
+        xyz="-8.02320899791198E-06 0.194762833402907 0.128888916941187"
+        rpy="0 0 0" />
+      <mass
+        value="1.10522962809227" />
+      <inertia
+        ixx="0.0225843178593198"
+        ixy="-7.27982747203185E-07"
+        ixz="-1.78485875318381E-07"
+        iyy="0.00152004282471311"
+        iyz="0.000623589021520354"
+        izz="0.0230428803086098" />
     </inertial>
     <visual>
@@ -149,5 +149,5 @@
         name="">
         <color
-          rgba="0.68627 0.68627 0.68627 1" />
+          rgba="0.792156862745098 0.819607843137255 0.933333333333333 1" />
       </material>
     </visual>
@@ -166,6 +166,6 @@
     type="revolute">
     <origin
-      xyz="-0.087 0.19 0"
-      rpy="0 0 0" />
+      xyz="0 0 0"
+      rpy="1.5708 0 0" />
     <parent
       link="elfin_link1" />
@@ -173,10 +173,10 @@
       link="elfin_link2" />
     <axis
-      xyz="-1 0 0" />
-    <limit
+      xyz="0 0 1" />
+     <limit
       lower="-2.35"
       upper="2.35"
-      effort="420"
-      velocity="1.57" />
+      effort="104"
+      velocity="1.27" />
   </joint>
   <link
@@ -184,15 +184,15 @@
     <inertial>
       <origin
-        xyz="0.067584 -0.041479 -1.1421E-05"
-        rpy="0 0 0" />
-      <mass
-        value="1.5324" />
-      <inertia
-        ixx="0.00514"
-        ixy="0.0014834"
-        ixz="-5.7782E-07"
-        iyy="0.0028926"
-        iyz="-3.0654E-07"
-        izz="0.0060883" />
+        xyz="0.0461694549854045 1.67843463302067E-05 -0.0210719533256843"
+        rpy="0 0 0" />
+      <mass
+        value="1.07590672952063" />
+      <inertia
+        ixx="0.00137807691049161"
+        ixy="-3.57302576480749E-07"
+        ixz="-0.00013179565326652"
+        iyy="0.00135308160804782"
+        iyz="9.02259193989242E-07"
+        izz="0.00154416453671479" />
     </inertial>
     <visual>
@@ -207,5 +207,5 @@
         name="">
         <color
-          rgba="0.86667 0.86667 0.8902 1" />
+          rgba="0.792156862745098 0.819607843137255 0.933333333333333 1" />
       </material>
     </visual>
@@ -225,5 +225,5 @@
     <origin
       xyz="0 0.455 0"
-      rpy="-3.1416 0 0" />
+      rpy="-3.1416 0 1.5708" />
     <parent
       link="elfin_link2" />
@@ -231,179 +231,63 @@
       link="elfin_link3" />
     <axis
-      xyz="1 0 0" />
+      xyz="0 0 1" />
     <limit
       lower="-2.61"
       upper="2.61"
-      effort="200"
-      velocity="1.57" />
-  </joint>
-  <link
-    name="elfin_link4">
-    <inertial>
-      <origin
-        xyz="-0.017434 -0.33294 -0.00015134"
-        rpy="0 0 0" />
-      <mass
-        value="0.5" />
-      <inertia
-        ixx="0.00542441"
-        ixy="0.0020749"
-        ixz="1.0501E-05"
-        iyy="0.014338"
-        iyz="-0.00041574"
-        izz="0.00607489" />
-    </inertial>
-    <visual>
-      <origin
-        xyz="0 0 0"
-        rpy="0 0 0" />
-      <geometry>
-        <mesh
-          filename="package://elfin_description/meshes/elfin5_l/elfin_link4.STL" />
-      </geometry>
-      <material
-        name="">
-        <color
-          rgba="0.68627 0.68627 0.68627 1" />
-      </material>
-    </visual>
-    <collision>
-      <origin
-        xyz="0 0 0"
-        rpy="0 0 0" />
-      <geometry>
-        <mesh
-          filename="package://elfin_description/meshes/elfin5_l/elfin_link4.STL" />
-      </geometry>
-    </collision>
-  </link>
-  <joint
-    name="elfin_joint4"
-    type="revolute">
-    <origin
-      xyz="0.087 -0.1255 0"
-      rpy="3.1416 0 0" />
-    <parent
-      link="elfin_link3" />
-    <child
-      link="elfin_link4" />
-    <axis
-      xyz="0 1 0" />
-    <limit
-      lower="-3.14"
-      upper="3.14"
-      effort="200"
-      velocity="1.57" />
-  </joint>
-  <link
-    name="elfin_link5">
-    <inertial>
-      <origin
-        xyz="-0.015972 -0.036591 1.4235E-06"
-        rpy="0 0 0" />
-      <mass
-        value="0.81192" />
-      <inertia
-        ixx="0.0018901"
-        ixy="0.00056728"
-        ixz="-4.2025E-08"
-        iyy="0.0010231"
-        iyz="5.0791E-09"
-        izz="0.002299" />
-    </inertial>
-    <visual>
-      <origin
-        xyz="0 0 0"
-        rpy="0 0 0" />
-      <geometry>
-        <mesh
-          filename="package://elfin_description/meshes/elfin5_l/elfin_link5.STL" />
-      </geometry>
-      <material
-        name="">
-        <color
-          rgba="0.79216 0.81961 0.93333 1" />
-      </material>
-    </visual>
-    <collision>
-      <origin
-        xyz="0 0 0"
-        rpy="0 0 0" />
-      <geometry>
-        <mesh
-          filename="package://elfin_description/meshes/elfin5_l/elfin_link5.STL" />
-      </geometry>
-    </collision>
-  </link>
-  <joint
-    name="elfin_joint5"
-    type="revolute">
-    <origin
-      xyz="0 0.3695 0"
-      rpy="-3.1416 0 0" />
-    <parent
-      link="elfin_link4" />
-    <child
-      link="elfin_link5" />
-    <axis
-      xyz="1 0 0" />
-    <limit
-      lower="-2.56"
-      upper="2.56"
       effort="69"
       velocity="1.57" />
   </joint>
   <link
-    name="elfin_link6">
-    <inertial>
-      <origin
-        xyz="-0.0072549 0.027062 3.208E-05"
-        rpy="0 0 0" />
-      <mass
-        value="0.11343" />
-      <inertia
-        ixx="7.4923E-05"
-        ixy="-2.3429E-06"
-        ixz="-1.8394E-07"
-        iyy="0.0001278"
-        iyz="-4.8092E-08"
-        izz="7.6653E-05" />
-    </inertial>
-    <visual>
-      <origin
-        xyz="0 0 0"
-        rpy="0 0 0" />
-      <geometry>
-        <mesh
-          filename="package://elfin_description/meshes/elfin5_l/elfin_link6.STL" />
-      </geometry>
-      <material
-        name="">
-        <color
-          rgba="0.77647 0.75686 0.73725 1" />
-      </material>
-    </visual>
-    <collision>
-      <origin
-        xyz="0 0 0"
-        rpy="0 0 0" />
-      <geometry>
-        <mesh
-          filename="package://elfin_description/meshes/elfin5_l/elfin_link6.STL" />
-      </geometry>
-    </collision>
-  </link>
-  <joint
-    name="elfin_joint6"
-    type="revolute">
-    <origin
-      xyz="0 -0.1065 0"
-      rpy="3.1416 0 0" />
-    <parent
-      link="elfin_link5" />
-    <child
-      link="elfin_link6" />
-    <axis
-      xyz="0 1 0" />
+    name="elfin_link4">
+    <inertial>
+      <origin
+        xyz="-2.52415186551188E-05 -0.0426485662035081 0.296130346848396"
+        rpy="0 0 0" />
+      <mass
+        value="0.773486357600959" />
+      <inertia
+        ixx="0.0065953698905962"
+        ixy="-7.26135070513294E-07"
+        ixz="2.7130632453124E-06"
+        iyy="0.00593057161737003"
+        iyz="0.00162601275838063"
+        izz="0.00175532385127571" />
+    </inertial>
+    <visual>
+      <origin
+        xyz="0 0 0"
+        rpy="0 0 0" />
+      <geometry>
+        <mesh
+          filename="package://elfin_description/meshes/elfin5_l/elfin_link4.STL" />
+      </geometry>
+      <material
+        name="">
+        <color
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